File: MIMO_SAR_RADAR.kicad_sch (KiCad schematic)
At the start: 131 parts, among them IC1 SKY13418-485LF, IC10 PSA2-6+, IC11 ADL5380ACPZ-R7, IC12 ADL5380ACPZ-R7, IC15 SKY13418-485LF, IC16 ADA4940-2ACPZ-RL, IC18 ADA4940-2ACPZ-RL, IC2 SKY13418-485LF, IC20 ADS8588SIPM, IC21 LMX2594RHAT, IC22 SKY13418-485LF, IC23 SKY13418-485LF, IC5 LT3042IMSE#PBF, IC6 PMA3-73-1W+, IC7 PSA2-6+, J1 Conn_01x06_Pin, J2 Conn_Coaxial_Small, J3 Conn_Coaxial_Small, Q1 D44VH10, U1 LM2596S-12, U2 STM32H7A3IGTx, U3 ESP32-C3-WROOM-02, U5 LM1117DT-3.3, Y1 SiT9121AI-2B1-33E100.000000G

Commit message: work...
Parts:
- removed C11, C12, C4, C5: C_Small, symbol Device:C_Small
- removed FL4: LFCN-6000+, LFCN6000, symbol RF_LP:LFCN-6000+
- removed FL8: HFCG-3000+, HFCG3000, symbol RF_HP:HFCG-3000+
- removed IC12: ADL5380ACPZ-R7, QFN50P400X400X100-25N, symbol RF_Modulators:ADL5380ACPZ-R7
- removed IC16: ADA4940-2ACPZ-RL, QFN50P400X400X80-25N-D, symbol ADC_DRIVER:ADA4940-2ACPZ-RL
- removed IC7: PSA2-6+, SOT65P215X100-6N, symbol LNA:PSA2-6+
- removed R11, R12, R4, R5: R_Small, symbol Device:R_Small
- added C59: 220uF, symbol Device:C_Small
- added C60, C63, C65: 0.1uF, symbol Device:C_Small
- added C61, C62, C64: 1uF, symbol Device:C_Small
- added D2, D3: SS54, symbol Device:D_Schottky
- added J4: Conn_01x02_Pin, Connector_AMASS:AMASS_XT60-F_1x02_P7.20mm_Vertical, symbol Connector:Conn_01x02_Pin
- added L4: 100uH, symbol Device:L_Small
- added R13, R7: 0R, symbol Device:R_Small
- added R8: 200R, symbol Device:R_Small
- added T1, T2: TCM1-63AX-2+, TCM163AX2, symbol Balun:TCM1-63AX-2+
- C14, C15: value C_Small -> 2400pF
- C58: value C_Small -> 680uF
- J3: footprint (none) -> Connector_Coaxial:SMA_Amphenol_132289_EdgeMount
- L2: value 8nH -> 8nH (experimental)
- L3: value L -> TCCH-80+
Connections:
- net +12V: now also R7.2; no longer U1.2 (OUT)
- net 5V_CLEAN: now also IC11.13 (VCC2), IC11.24 (VDD3), IC11.6 (VCC1), C60.2, C61.2, C62.2, C63.2, C64.2, C65.2, R8.2
- net GND: now also IC11.1 (GND3_2), IC11.11 (GND4), IC11.14 (GND2_2), IC11.17 (GND2), IC11.18 (GND3_3), IC11.2 (GND1_2), IC11.20 (GND3_4), IC11.23 (GND3), IC11.5 (GND1), IC11.8 (GND4_2), C59.2, C60.1, C61.1, C62.1, C63.1, C64.1, C65.1, D2.2 (A), J4.1 (Pin_1), R13.1
- net at IC11.19 (ADJ): now also R8.1
- net at IC11.7 (ENBL): now also R13.2
- net at C58.1, U1.1 (VIN): now also D3.1 (K)
- net at U1.4 (FB): now also C59.1, L4.2, R7.1
- new net: D3.2 (A), J4.2 (Pin_2)
- new net: D2.1 (K), L4.1, U1.2 (OUT)
Other:
- moved on the sheet: C1, C10, C14, C15, C16, C3, C57, C9, FL1, FL7, IC1, IC10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

Commit message: RX chain improvements and negative supply
Parts:
- removed IC18: ADA4940-2ACPZ-RL, QFN50P400X400X80-25N-D, symbol ADC_DRIVER:ADA4940-2ACPZ-RL
- removed IC20: ADS8588SIPM, QFP50P1200X1200X160-64N, symbol HS_ADCS:ADS8588SIPM
- removed R10, R9: R_Small, symbol Device:R_Small
- added C11, C12, C4, C5: 100pF, symbol Device:C_Small
- added C66, C67, C68, C69, C70, C71: C_Small, symbol Device:C_Small
- added IC3: ADS8584SIPM, QFP50P1200X1200X160-64N, symbol 4CH_ADC:ADS8584SIPM
- added IC4, IC7: OPA1632DGNR, SOP65P490X110-9N, symbol DIFF_AMPS:OPA1632DGNR
- added IC8: LMX2594RHAT, QFN50P600X600X100-41N-D, symbol LMX94:LMX2594RHAT
- added L10, L11, L12, L13, L14, L15, L16, L5, L6, L7, L8, L9: L_Small, symbol Device:L_Small
- added R4: 500R, symbol Device:R_Small
- added R5: R_Small, symbol Device:R_Small
- C1, C10, C3, C9: value C_Small -> 10uF
- C61, C62, C64: value 1uF -> 100pF
- R1: value R_Small -> 500R
Connections:
- net 5V_CLEAN: now also R3.2, R5.1
- net GND: now also T1.2 (PRIMARY/GND), T2.2 (PRIMARY/GND), IC4.2 (VOCM), IC4.9 (EP), IC7.2 (VOCM), IC7.9 (EP); no longer C1.1, C10.1, C3.1, C9.1
- net at R1.2: now also C69.2, IC4.1 (VIN-), L10.2; no longer C1.2
- net at C9.2: now also L8.1
- net at C10.2: now also L5.1
- net at IC11.10 (LOIN): now also C11.1
- net at IC11.15 (QLO): now also C3.1
- net at IC11.16 (QHI): now also C1.1
- net at IC11.21 (REFIN): now also C5.1
- net at IC11.22 (REFIP): now also C4.1
- net IHI1: now reaches IC11.3 (IHI)
- net IHI1: now also C10.1
- net ILO1: now reaches IC11.4 (ILO)
- net ILO1: now also C9.1
- net at IC11.9 (LOIP): now also C12.1
- net RX1_BALUN_IN: now reaches T2.3 (PRIMARY_DOT)
- net RX1_BALUN_IN: now also C15.2
- net at T2.4 (SECONDARY): now also C5.2
- net at T2.6 (SECONDARY_DOT): now also C4.2
- net at R3.1: now also IC7.7 (ENABLE)
- net at C3.2: now also L14.1; no longer R3.2
- net SPLIT_TX: now reaches TDK_HHM2952A1/auf_PCB1.2 (Coupled)
- net SPLIT_TX: now also T1.3 (PRIMARY_DOT)
- net at R1.1: now also C69.1, IC4.8 (VIN+), L7.2
- net at T1.4 (SECONDARY): now also C11.2
- net at T1.6 (SECONDARY_DOT): now also C12.2
- new net: IC4.7 (ENABLE), R5.2
- new net: C67.1, L12.2, L13.1
- new net: C67.2, L15.2, L16.1
- new net: C66.1, IC7.8 (VIN+), L13.2, R4.1
- new net: C66.2, IC7.1 (VIN-), L16.2, R4.2
- new net: C68.2, L14.2, L15.1
- new net: C68.1, L11.2, L12.1
- new net: C71.1, L5.2, L6.1
- new net: C71.2, L8.2, L9.1
- new net: C70.1, L6.2, L7.1
- new net: C70.2, L10.1, L9.2
- new net: C1.2, L11.1
Other:
- note added: "450 Ω differential load on I and Q outputs at 900 MHz 6.9 dB 200 Ω differential load on I and Q outputs at 900 MHz"
- note added: "Sollte zwischen -6dbm und 6dbm liegen (evtl rf limiter verbauen..)"
- note removed: "RC TIEFPASS (Anitaliasing )"
- moved on the sheet: C45, C46, C47, C48, C49, C50, C51, C52, C53, C54, C55, C56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

Commit message: Structure +2.nd rx channel
Parts:
- removed IC2: SKY13418-485LF, SKY13418485LF, symbol SKY13:SKY13418-485LF
- removed IC8: LMX2594RHAT, QFN50P600X600X100-41N-D, symbol LMX94:LMX2594RHAT
- added C72, C75: 2400pF, symbol Device:C_Small
- added C73: 0.01uF, Capacitor_SMD:C_0603_1608Metric, symbol Device:C_Small
- added C74: 0.1uF, Capacitor_SMD:C_0603_1608Metric, symbol Device:C_Small
- added C76, C78, C80, C81, C82, C83, C85: 100pF, symbol Device:C_Small
- added C77, C79, C84: 0.1uF, symbol Device:C_Small
- added C86, C87, C88, C89: 10uF, symbol Device:C_Small
- added C90, C91, C92, C93, C94, C95: C_Small, symbol Device:C_Small
- added FL2: LFCN-6000+, LFCN6000, symbol RF_LP:LFCN-6000+
- added FL8: HFCG-3000+, HFCG3000, symbol RF_HP:HFCG-3000+
- added IC12: PSA2-6+, SOT65P215X100-6N, symbol LNA:PSA2-6+
- added IC13: ADL5380ACPZ-R7, QFN50P400X400X100-25N, symbol RF_Modulators:ADL5380ACPZ-R7
- added IC14, IC9: OPA1632DGNR, SOP65P490X110-9N, symbol DIFF_AMPS:OPA1632DGNR
- added IC8: SKY13418-485LF, SKY13418485LF, symbol SKY13:SKY13418-485LF
- added J5: SWD_CON, symbol Connector:Conn_01x05_Pin
- added L17: TCCH-80+, symbol Device:L
- added L18, L19, L20, L21, L22, L23, L24, L25, L26, L27, L28, L29: L_Small, symbol Device:L_Small
- added PS2: LM27762DSSR, SON50P200X300X80-13N-D, symbol LM27762DSSR:LM27762DSSR
- added R10: 200R, symbol Device:R_Small
- added R11, R12: 500R, symbol Device:R_Small
- added R14: 0R, symbol Device:R_Small
- added R15, R16: R_Small, symbol Device:R_Small
- added R9: 93.1R, Resistor_SMD:R_0805_2012Metric, symbol Device:R_Small
- added T3, T4: TCM1-63AX-2+, TCM163AX2, symbol Balun:TCM1-63AX-2+
- J4: footprint Connector_AMASS:AMASS_XT60-F_1x02_P7.20mm_Vertical -> Connector_AMASS:AMASS_XT60-M_1x02_P7.20mm_Vertical
Connections:
- net +3.3V: now also IC8.4 (VDD)
- net 5V_CLEAN: now also C74.2, C76.2, C77.2, C78.2, C79.2, C84.2, C85.2, IC13.13 (VCC2), IC13.24 (VDD3), IC13.6 (VCC1), R10.2, R15.2, R16.1, R9.2
- net GND: now also C73.1, C74.1, C76.1, C77.1, C78.1, C79.1, C84.1, C85.1, FL2.2 (GROUND_1), FL2.4 (GROUND_2), FL8.2 (GROUND_1), FL8.4 (GROUND_2), FL8.5 (GROUND_3), FL8.6 (GROUND_4), IC12.2 (GND_1), IC12.3 (GND_2), IC12.5 (GND_3), IC12.6 (GND_4), IC13.1 (GND3_2), IC13.11 (GND4), IC13.14 (GND2_2), IC13.17 (GND2), IC13.18 (GND3_3), IC13.2 (GND1_2), IC13.20 (GND3_4), IC13.23 (GND3), IC13.5 (GND1), IC13.8 (GND4_2), IC14.2 (VOCM), IC14.9 (EP), IC8.15 (GND), IC9.2 (VOCM), IC9.9 (EP), PS2.13 (PAD), PS2.4 (GND), R14.1, T3.2 (PRIMARY/GND), T4.2 (PRIMARY/GND)
- net IHI1: now also C86.1, IC13.3 (IHI)
- net ILO1: now also C87.1, IC13.4 (ILO)
- net RX1_BALUN_IN: now also C75.2, T3.3 (PRIMARY_DOT)
- net SPLIT_TX: now also T4.3 (PRIMARY_DOT)
- new net: C94.1, IC14.8 (VIN+), L26.2, R11.1
- new net: C94.2, IC14.1 (VIN-), L27.2, R11.2
- new net: IC13.19 (ADJ), R10.1
- new net: C92.1, L22.2, L26.1
- new net: IC13.7 (ENBL), R14.2
- new net: C86.2, L18.1
- new net: C83.1, IC13.10 (LOIN)
- new net: C89.1, IC13.15 (QLO)
- new net: C88.1, IC13.16 (QHI)
- new net: C81.1, IC13.21 (REFIN)
- new net: C80.1, IC13.22 (REFIP)
- new net: C82.1, IC13.9 (LOIP)
- new net: C87.2, L19.1
- new net: C75.1, IC12.4 (RF-OUT_&_VD), L17.2
- new net: IC14.7 (ENABLE), R16.2
- new net: C88.2, L20.1
- new net: C93.1, L24.2, L28.1
- new net: C95.1, IC9.8 (VIN+), L28.2, R12.1
- new net: FL2.1 (RF_IN), IC8.13 (ANT)
- new net: C73.2, L17.1, R9.1
- new net: FL2.3 (RF_OUT), FL8.1 (INPUT)
- new net: C72.1, FL8.3 (OUTPUT)
- new net: C72.2, IC12.1 (RF-IN)
- new net: C95.2, IC9.1 (VIN-), L29.2, R12.2
- new net: C90.2, L19.2, L23.1
- new net: C92.2, L23.2, L27.1
- new net: C83.2, T4.4 (SECONDARY)
- new net: C93.2, L25.2, L29.1
- new net: IC9.7 (ENABLE), R15.1
- new net: C81.2, T3.4 (SECONDARY)
- new net: C80.2, T3.6 (SECONDARY_DOT)
- new net: C91.1, L20.2, L24.1
- new net: C91.2, L21.2, L25.1
- new net: C90.1, L18.2, L22.1
- new net: C89.2, L21.1
- new net: C82.2, T4.6 (SECONDARY_DOT)
Other:
- note added: "ANTENNA SIDE"
- note added: "MCU"
- note added: "RX"
- note added: "Supply"
- note added: "TX"
- moved on the sheet: C13, C17, C18, C19, C2, C20, C21, C22, C23, C24, C25, C26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

Commit message: better adc, easyer rx chain design
Parts:
- removed IC14, IC4, IC7, IC9: OPA1632DGNR, SOP65P490X110-9N, symbol DIFF_AMPS:OPA1632DGNR
- removed IC3: ADS8584SIPM, QFP50P1200X1200X160-64N, symbol 4CH_ADC:ADS8584SIPM
- removed PS2: LM27762DSSR, SON50P200X300X80-13N-D, symbol LM27762DSSR:LM27762DSSR
- removed R15, R16: R_Small, symbol Device:R_Small
- added C96, C97, C98: 1uF, symbol Device:C_Small
- added C99: C_Small, symbol Device:C_Small
- added IC2: AD7380-4BCPZ, QFN50P400X400X60-25N-D, symbol AD7380:AD7380-4BCPZ
- Q1: footprint (none) -> Package_TO_SOT_THT:TO-220-3_Horizontal_TabDown
Connections:
- net +3.3V: now also R3.1, C96.1, IC2.4 (VCC)
- net 5V_CLEAN: no longer R3.2, R5.1
- net GND: now also R5.2, C96.2, C97.1, C98.2, C99.2, IC2.1 (GND_1), IC2.14 (GND_3), IC2.16 (GND_4), IC2.25 (EP), IC2.5 (GND_2)
- net IHI1: no longer C86.1, IC13.3 (IHI)
- net ILO1: no longer C87.1, IC13.4 (ILO)
- net RX1_BALUN_IN: no longer C75.2, T3.3 (PRIMARY_DOT)
- net ADC_C+: now reaches C94.1, L26.2, R11.1
- net ADC_C+: now also IC2.9 (AINC+)
- net ADC_C-: now reaches C94.2, L27.2, R11.2
- net ADC_C-: now also IC2.8 (AINC-)
- net ADC_A-: now reaches C69.2, L10.2, R1.2
- net ADC_A-: now also IC2.12 (AINA-)
- net ADC_A+: now reaches C69.1, L7.2, R1.1
- net ADC_A+: now also IC2.13 (AINA+)
- net ADC_B+: now reaches C66.1, L13.2, R4.1
- net ADC_B+: now also IC2.11 (AINB+)
- net ADC_B-: now reaches C66.2, L16.2, R4.2
- net ADC_B-: now also IC2.10 (AINB-)
- net ADC_D+: now reaches C95.1, L28.2, R12.1
- net ADC_D+: now also IC2.7 (AIND+)
- net ADC_D-: now reaches C95.2, L29.2, R12.2
- net ADC_D-: now also IC2.6 (AIND-)
- new net: C99.1, IC2.17 (REFIO), R3.2, R5.1
- new net: C97.2, IC2.3 (REGCAP)
- new net IHI2: C86.1, IC13.3 (IHI)
- new net ILO2: C87.1, IC13.4 (ILO)
- new net RX2_BALUN_IN: C75.2, T3.3 (PRIMARY_DOT)
- new net VCC: C98.1, IC2.2 (VLOGIC)
- no-connect marks 3 -> 4
Other:
- note added: "Oder lieber single ended?"

Commit message: new mcu , swd interface
Parts:
- removed U2: STM32H7A3IGTx, Package_QFP:LQFP-176_24x24mm_P0.5mm, symbol MCU_ST_STM32H7:STM32H7A3IGTx
- added J6: SWD, Connector_JST:JST_XH_B4B-XH-A_1x04_P2.50mm_Vertical, symbol Connector:Conn_01x04_Pin
- added U4: STM32H745IITx, Package_QFP:LQFP-176_24x24mm_P0.5mm, symbol MCU_ST_STM32H7:STM32H745IITx
- renumbered HMC476MP86(FREQUENZBEREICH)1 to HMC476MP86(FREQUENZBEREICH)(nichtkomplettnotwendig)
Connections:
- net +3.3V: now also U4.105 (VDD), U4.113 (VDD), U4.121 (VDD33_USB), U4.126 (VDD), U4.13 (VDD), U4.136 (VDD), U4.152 (VDD), U4.16 (VDDSMPS), U4.160 (VDD), U4.176 (VDD), U4.25 (VDD), U4.44 (VDD), U4.48 (VDD), U4.65 (VDD), U4.7 (VDD), U4.71 (VDD), U4.84 (VDD), U4.92 (VDD), U4.99 (VDD)
- net GND: now also J6.3 (Pin_3)
- new net: U4.100 (VSS), U4.106 (VSS), U4.112 (VSS), U4.119 (VSS), U4.12 (VSS), U4.134 (VSS), U4.137 (VSS), U4.151 (VSS), U4.159 (VSS), U4.173 (VSS), U4.24 (VSS), U4.45 (VSS), U4.47 (VSS), U4.6 (VSS), U4.64 (VSS), U4.70 (VSS), U4.81 (VSS), U4.83 (VSS), U4.93 (VSS)
- new net SWCLK: J6.2 (Pin_2), U4.138 (PA14)
- new net SWD_IO: J6.4 (Pin_4), U4.132 (PA13)

Commit message: mcu interfaces
Parts:
- removed IC1, IC8: SKY13418-485LF, SKY13418485LF, symbol SKY13:SKY13418-485LF
- removed J5: SWD_CON, symbol Connector:Conn_01x05_Pin
- added C100: C_Small, symbol Device:C_Small
- added C101: 4.7uF, Capacitor_SMD:C_0603_1608Metric, symbol Device:C_Small
- added C102, C104: 10uF, Capacitor_SMD:C_0805_2012Metric, symbol Device:C_Small
- added C103: 220pF, Capacitor_SMD:C_0603_1608Metric, symbol Device:C_Small
- added C105: 100nF, symbol Device:C_Small
- added C106: 4.7uF, symbol Device:C_Small
- added C107: 2.2uF, symbol Device:C_Small
- added J5, J8: Conn_Coaxial_Small, Connector_Coaxial:SMA_Amphenol_132289_EdgeMount, symbol Connector:Conn_Coaxial_Small
- added J7: Conn_01x06_Pin, Connector_JST:JST_PH_B6B-PH-K_1x06_P2.00mm_Vertical, symbol Connector:Conn_01x06_Pin
- added L30: 2.2uH, Inductor_SMD:L_0805_2012Metric_Pad1.15x1.40mm_HandSolder, symbol Device:L_Small
- added R15, R43: 10k, symbol Device:R_Small
- added R16: inf, symbol Device:R_Small
- added SW1: SW_Push, symbol Switch:SW_Push
Connections:
- net CLOCK is gone; now on net CLOCK_VCO: IC21.16 (SCK)
- net MOSI is gone; now on net MOSI_VCO: IC21.17 (SDI)
- net SS is gone; now on net SS_VCO: IC21.24 (CSB)
- net +3.3V: now also J6.1 (Pin_1), U4.39 (VREF+), U4.40 (VDDA), C101.1, C105.1, C106.1, C107.1, J7.2 (Pin_2), R16.1, R43.1; no longer U4.121 (VDD33_USB)
- net GND: now also U4.100 (VSS), U4.106 (VSS), U4.112 (VSS), U4.119 (VSS), U4.12 (VSS), U4.134 (VSS), U4.137 (VSS), U4.14 (VSSSMPS), U4.151 (VSS), U4.159 (VSS), U4.173 (VSS), U4.24 (VSS), U4.38 (VSSA), U4.45 (VSS), U4.47 (VSS), U4.6 (VSS), U4.64 (VSS), U4.70 (VSS), U4.81 (VSS), U4.83 (VSS), U4.93 (VSS), C100.1, C101.2, C102.2, C103.2, C104.2, C105.2, C106.2, C107.2, J5.2 (Ext), J7.1 (Pin_1), J8.2 (Ext), R15.2, SW1.2
- net RF_SWITCH_BIT_0: now also U4.55 (PB0), J7.3 (Pin_3)
- net RF_SWITCH_BIT_1: now also U4.56 (PB1), J7.4 (Pin_4)
- net RF_SWITCH_BIT_2: now also U4.57 (PB2), J7.5 (Pin_5)
- net RF_SWITCH_BIT_3: now also U4.162 (PB3), J7.6 (Pin_6)
- net at FL1.1 (RF_IN): now also J5.1 (In)
- net at FL2.1 (RF_IN): now also J8.1 (In)
- net SDOA: now reaches U4.122 (PC6)
- net SDOA: now also IC2.19 (SDOA)
- net SDOB: now reaches U4.123 (PC7)
- net SDOB: now also IC2.20 (SDOB)
- net SDOC: now reaches U4.124 (PC8)
- net SDOC: now also IC2.23 (SDOC)
- net SDOD: now reaches U4.125 (PC9)
- net SDOD: now also IC2.24 (SDOD/~{ALERT})
- net VCAP: now reaches U4.133 (VCAP)
- net VCAP: now also U4.135 (VDDLDO), U4.17 (VFBSMPS), U4.172 (VCAP), U4.175 (VDDLDO), U4.80 (VCAP), U4.82 (VDDLDO), C102.1, C104.1, L30.1
- net VLXSMPS: now reaches U4.15 (VLXSMPS)
- net VLXSMPS: now also C103.1, L30.2
- net BOOT0: now reaches U4.167 (BOOT0)
- net BOOT0: now also R15.1, R16.2
- net at U4.174 (PDR_ON): now also R43.2
- net NRST: now reaches U4.33 (NRST)
- net NRST: now also C100.2, SW1.1
- net RX1_SWITCH_BIT_0: now reaches U4.34 (PC0)
- net RX1_SWITCH_BIT_1: now reaches U4.35 (PC1)
- net RX1_SWITCH_BIT_2: now reaches U4.36 (PC2_C)
- net RX1_SWITCH_BIT_3: now reaches U4.37 (PC3_C)
- net SS_VCO: now reaches U4.49 (PA4)
- net CLOCK_VCO: now reaches U4.50 (PA5)
- net MOSI_VCO: now reaches U4.52 (PA7)
- net CSNOT: now reaches IC2.18 (~{CS})
- net SDI_ADC: now reaches IC2.21 (SDI)
- net SCLK_ADC: now reaches IC2.22 (SCLK)
Other:
- note added: "PULL HIGH FOR USB BOOTING"
- note added: "STM_ADC-TEST"
- moved on the sheet: J6, U3, U4

Commit message: finishing up schematic
Parts:
- added J10, J9: Conn_01x06_Pin, Connector_JST:JST_PH_B6B-PH-K_1x06_P2.00mm_Vertical, symbol Connector:Conn_01x06_Pin
- added R2, R44, R45, R7: R_Small, symbol Device:R_Small
- R3: renamed from R16; now not fitted
- renumbered C107 to C1, C37 to C10, C69 to C100, C66 to C101, C94 to C102, C95 to C103, C97 to C104, C96 to C105, C99 to C106, C98 to C107, C38 to C11, C22 to C12, C28 to C13, C26 to C14, C20 to C15, C24 to C16, C18 to C17, C23 to C18, C29 to C19, C105 to C2, C27 to C20, C25 to C22, C19 to C23, C17 to C24, C59 to C25, C31 to C26, C32 to C27, C33 to C28, C35 to C29, C106 to C3, C40 to C30, C50 to C31, C34 to C32, C43 to C33, C42 to C34, C36 to C35, C39 to C36, C30 to C37, C55 to C38, C44 to C39, C100 to C4, C41 to C40, C8 to C41, C51 to C42, C56 to C43, C53 to C44, C52 to C45, C6 to C46, C14 to C47, C72 to C48, C2 to C49, C101 to C5, C54 to C50, C13 to C51, C45 to C52, C7 to C53, C46 to C54, C57 to C55, C73 to C56, C16 to C57, C15 to C58, C74 to C59, C102 to C6, C75 to C60, C62 to C61, C63 to C62, C76 to C63, C77 to C64, C64 to C65, C65 to C66, C47 to C67, C78 to C68, C79 to C69, C103 to C7, C4 to C70, C5 to C71, C12 to C72, C11 to C73, C80 to C74, C81 to C75, C48 to C76, C82 to C77, C83 to C78, C60 to C79, C104 to C8, C49 to C80, C61 to C81, C84 to C82, C85 to C83, C10 to C84, C9 to C85, C1 to C86, C3 to C87, C86 to C88, C87 to C89, C58 to C9, C88 to C90, C89 to C91, C71 to C92, C68 to C93, C90 to C94, C91 to C95, C70 to C96, C67 to C97, C92 to C98, C93 to C99, D3 to D1, D1 to D3, FL7 to FL3, FL8 to FL4, FL9 to FL5, FL10 to FL6, HMC476MP86(FREQUENZBEREICH)(nichtkomplettnotwendig) to HMC476MP86(FREQUENZBEREICH)(nichtkomplettnotwendig)1, IC23 to IC1, IC13 to IC10, IC2 to IC11, IC15 to IC2, IC22 to IC3, IC21 to IC4, IC10 to IC6, IC12 to IC7, IC6 to IC8, IC11 to IC9, J2 to J1, J1 to J2, J6 to J3, J8 to J6, J3 to J8, L30 to L1, L14 to L10, L18 to L11, L19 to L12, L20 to L13, L21 to L14, L6 to L15, L9 to L16, L12 to L17, L15 to L18, L22 to L19, L4 to L2, L23 to L20, L24 to L21, L25 to L22, L7 to L23, L10 to L24, L13 to L25, L16 to L26, L26 to L27, L27 to L28, L28 to L29, L2 to L3, L29 to L30, L3 to L4, L17 to L5, L1 to L6, L5 to L7, L11 to L9, R43 to R1, R23 to R10, R22 to R11, R19 to R12, R21 to R13, R18 to R14, R25 to R15, R17 to R16, R26 to R17, R7 to R18, R24 to R19, R27 to R20, R36 to R21, R39 to R22, R2 to R23, R37 to R24, R38 to R25, R31 to R26, R6 to R27, R33 to R28, R9 to R30, R30 to R31, R13 to R33, R14 to R34, R34 to R35, R8 to R36, R10 to R37, R35 to R38, R42 to R39, R15 to R4, R1 to R40, R4 to R41, R11 to R42, R12 to R43, R3 to R46, R5 to R47, R40 to R5, R41 to R6, R28 to R8, R20 to R9, T2 to T1, T1 to T2, U4 to U1, U3 to U2, U1 to U3, U5 to U4
Connections:
- net +3.3V: now also J10.2 (Pin_2), J9.2 (Pin_2)
- net ADC_C+: now also R2.1
- net ADC_C-: now also R45.1
- net ADC_D+: now also R7.1
- net ADC_D-: now also R44.1
- net CSNOT: now also U1.85 (PB12)
- net GND: now also J10.1 (Pin_1), J9.1 (Pin_1), R44.2, R45.2
- net RX1_SWITCH_BIT_0: now also J10.3 (Pin_3)
- net RX1_SWITCH_BIT_1: now also J10.4 (Pin_4)
- net RX1_SWITCH_BIT_2: now also J10.5 (Pin_5)
- net RX1_SWITCH_BIT_3: now also J10.6 (Pin_6)
- net SCLK_ADC: now also U1.86 (PB13)
- net SDI_ADC: now also U1.88 (PB15)
- net SDOA: now also U1.87 (PB14)
- net RX2_SWITCH_BIT_0: now reaches U1.143 (PD0)
- net RX2_SWITCH_BIT_0: now also J9.3 (Pin_3)
- net RX2_SWITCH_BIT_1: now reaches U1.144 (PD1)
- net RX2_SWITCH_BIT_1: now also J9.4 (Pin_4)
- net RX2_SWITCH_BIT_2: now reaches U1.145 (PD2)
- net RX2_SWITCH_BIT_2: now also J9.5 (Pin_5)
- net RX2_SWITCH_BIT_3: now reaches U1.146 (PD3)
- net RX2_SWITCH_BIT_3: now also J9.6 (Pin_6)
- net at U1.21 (PF3): now also R2.2
- net at U1.42 (PA1): now also R7.2
Other:
- moved on the sheet: U2

Commit message: efficiency boost
Parts:
- removed C38: 10uF, symbol Device:C_Small
- removed C43: 100uF, symbol Device:C_Small
- removed U4: LM1117DT-3.3, Package_TO_SOT_SMD:TO-252-3_TabPin2, symbol Regulator_Linear:LM1117DT-3.3
- added C108: 220uF, symbol Device:C_Small
- added C109: 680uF, symbol Device:C_Small
- added D4: SS54, symbol Device:D_Schottky
- added L31: 100uH, symbol Device:L_Small
- added R48: 0R, symbol Device:R_Small
- added U5: LM2596S-3.3, Package_TO_SOT_SMD:TO-263-5_TabPin3, symbol Regulator_Switching:LM2596S-3.3
Connections:
- net +3.3V: now also R48.2
- net GND: now also C108.2, C109.2, D4.2 (A), U5.5 (~{ON}/OFF)
- net at C9.1, D1.1 (K), U3.1 (VIN): now also C109.1, U5.1 (VIN)
- new net: C108.1, L31.2, R48.1, U5.4 (FB)
- new net: D4.1 (K), L31.1, U5.2 (OUT)
Other:
- moved on the sheet: C25, C31, C42, C44, C45, C50, C52, C54, C67, C76, C80, C9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
