File: MIMO_SAR_RADAR.kicad_sch (KiCad schematic)
At the start: 231 parts, among them IC1 SKY13418-485LF, IC10 ADL5380ACPZ-R7, IC11 AD7380-4BCPZ, IC2 SKY13418-485LF, IC3 SKY13418-485LF, IC4 LMX2594RHAT, IC5 LT3042IMSE#PBF, IC6 PSA2-6+, IC7 PSA2-6+, IC8 PMA3-73-1W+, IC9 ADL5380ACPZ-R7, J1 Conn_Coaxial_Small, J10 Conn_01x06_Pin, J2 Conn_01x06_Pin, J3 SWD, J4 Conn_01x02_Pin, J5 Conn_Coaxial_Small, J6 Conn_Coaxial_Small, J7 Conn_01x06_Pin, J8 Conn_Coaxial_Small, J9 Conn_01x06_Pin, Q1 D44VH10, SW1 SW_Push, T1 TCM1-63AX-2+, T2 TCM1-63AX-2+, T3 TCM1-63AX-2+, T4 TCM1-63AX-2+, U1 STM32H745IITx, U2 ESP32-C3-WROOM-02, U3 LM2596S-12, U5 LM2596S-3.3, Y1 SiT9121AI-2B1-33E100.000000G

Commit message: battery system angefangen
Parts:
- removed C109: 680uF, symbol Device:C_Small
- added BT1: Battery_Cell, Battery:BatteryHolder_Keystone_1042_1x18650, symbol Device:Battery_Cell
- added C38: 10uF, symbol Device:C_Small
- added C43: 680uF, Capacitor_SMD:C_Elec_10x10.2, symbol Device:C_Small
- added R49: R_Small, symbol Device:R_Small
- C9: footprint (none) -> Capacitor_SMD:C_Elec_10x10.2
Connections:
- net +3.3V: now also U2.1 (3V3), C38.1, R49.1
- net GND: now also C38.2, C43.2
- net at C9.1, D1.1 (K), U3.1 (VIN)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: now also C43.1
- net at U1.150 (PD7): now also U2.16 (IO2)
- net at U2.2 (EN): now also R49.2
Other:
- moved on the sheet: U2

Commit message: layout
Parts:
- removed BT1: Battery_Cell, Battery:BatteryHolder_Keystone_1042_1x18650, symbol Device:Battery_Cell
- removed C25: 220uF, symbol Device:C_Small
- removed C43, C9: 680uF, Capacitor_SMD:C_Elec_10x10.2, symbol Device:C_Small
- removed D1, D2, D4: SS54, symbol Device:D_Schottky
- removed L2, L31: 100uH, symbol Device:L_Small
- removed L3: 8nH (experimental), symbol Device:L
- removed L4, L5: TCCH-80+, symbol Device:L
- removed R18, R26, R48: 0R, symbol Device:R_Small
- removed U3: LM2596S-12, Package_TO_SOT_SMD:TO-263-5_TabPin3, symbol Regulator_Switching:LM2596S-12
- removed U5: LM2596S-3.3, Package_TO_SOT_SMD:TO-263-5_TabPin3, symbol Regulator_Switching:LM2596S-3.3
- added C109, C119: 4.7uF, Capacitor_SMD:C_0603_1608Metric, symbol Device:C_Small
- added C110, C120: C_Small, Capacitor_SMD:C_0603_1608Metric, symbol Device:C_Small
- added C111, C113, C117, C121, C123: 10uF, Capacitor_SMD:C_0603_1608Metric, symbol Device:C_Small
- added C112, C122: 0.47pF, Capacitor_SMD:C_0603_1608Metric, symbol Device:C_Small
- added C114: 3.3nF, Capacitor_SMD:C_0603_1608Metric, symbol Device:C_Small
- added C115: 22uF, Capacitor_SMD:C_0805_2012Metric, symbol Device:C_Small
- added C116: 0.1uF, Capacitor_SMD:C_0603_1608Metric, symbol Device:C_Small
- added D1: SMF18A, Diode_SMD:D_SMF, symbol Diode:SMF18A
- added D4: VCO_POWER_CHECK, LED_SMD:LED_0603_1608Metric, symbol Device:LED
- added D5: SS54, Diode_SMD:D_SMA, symbol Device:D_Schottky
- added H1, H2, H3: MountingHole, MountingHole:MountingHole_3.2mm_M3_DIN965_Pad, symbol Mechanical:MountingHole
- added IC12, IC14: LT3042IMSE#PBF, Low_noise_LDO:SOP50P490X110-11N, symbol Low_noise_LDO:LT3042IMSE#PBF
- added L2, L4, L5: TCCH-80, TCCH-80:GU1604, symbol TCCH:TCCH-80
- added L31: XFL4020-222MEB, XFL4020-222:XFL4020-222ME, symbol XFL4020-222:XFL4020-222MEB
- added PS2: TPS62150RGTR, TPS62150:QFN50P300X300X100-17N-D, symbol TPS62150:TPS62150RGTR
- added Q2: DPAK, Package_TO_SOT_SMD:TO-252-2, symbol Simulation_SPICE:NPN
- added Q4: D44VH10, Package_TO_SOT_SMD:TO-252-2, symbol Simulation_SPICE:NPN
- added R50, R58: 10k, Resistor_SMD:R_0603_1608Metric, symbol Device:R_Small
- added R51: 121k, Resistor_SMD:R_0603_1608Metric, symbol Device:R_Small
- added R52, R60: 249k, Resistor_SMD:R_0603_1608Metric, symbol Device:R_Small
- added R53, R61: 49k, Resistor_SMD:R_0603_1608Metric, symbol Device:R_Small
- added R54: 180k, Resistor_SMD:R_0603_1608Metric, symbol Device:R_Small
- added R55: 562k, Resistor_SMD:R_0603_1608Metric, symbol Device:R_Small
- added R56, R62, R63, R64: 0R, Resistor_SMD:R_0603_1608Metric, symbol Device:R_Small
- added R57: R_Small, Resistor_SMD:R_0603_1608Metric, symbol Device:R_Small
- added R59: 33k, Resistor_SMD:R_0603_1608Metric, symbol Device:R_Small
- added SW2: SW_Push, symbol Switch:SW_Push
- C1, C104, C105, C106, C107, C12, C13, C14, C15, C16, C17, C18, C19, C2, C20, C21, C22, C23, C26, C29, C3, C30, C31, C32, C35, C36, C37, C4, C40, C42, C44, C45, C46, C48, C49, C50, C52, C53, C54, C61, C62, C63, C64, C65, C66, C68, C69, C76, C79, C80, C81, C82, C83: footprint (none) -> Capacitor_SMD:C_0603_1608Metric
- C10, C100, C101, C102, C103, C11, C24, C27, C28, C33, C34, C39, C47, C58, C60, C70, C71, C72, C73, C74, C75, C77, C78, C84, C85, C86, C87, C88, C89, C90, C91, C92, C93, C94, C95, C96, C97, C98, C99: footprint (none) -> Capacitor_SMD:C_0402_1005Metric
- C108: value 220uF -> 10uF; footprint (none) -> Capacitor_SMD:C_0603_1608Metric
- C38, C67: footprint (none) -> Capacitor_SMD:C_0805_2012Metric
- D3: footprint (none) -> LED_SMD:LED_0603_1608Metric
- FL1, FL2, FL5: footprint LFCN6000 -> RF_LP:LFCN6000
- FL3, FL4, FL6: footprint HFCG3000 -> RF_HP:HFCG3000
- HMC476MP86(FREQUENZBEREICH)(nichtkomplettnotwendig)1: footprint ERA3 -> ERA-3+:ERA3
- IC1, IC2, IC3: footprint SKY13418485LF -> SKY13:SKY13418485LF
- IC10, IC9: footprint QFN50P400X400X100-25N -> RF_Modulators:QFN50P400X400X100-25N
- IC11: footprint QFN50P400X400X60-25N-D -> AD7380:QFN50P400X400X60-25N-D
- IC4: footprint QFN50P600X600X100-41N-D -> Package_DFN_QFN:QFN-40-1EP_6x6mm_P0.5mm_EP4.6x4.6mm
- IC5: footprint SOP50P490X110-11N -> Low_noise_LDO:SOP50P490X110-11N
- IC6, IC7: footprint SOT65P215X100-6N -> LNA:SOT65P215X100-6N
- IC8: footprint QFN51P300X300X89-13N -> PMA3:QFN51P300X300X89-13N
- J1: footprint (none) -> Connector_Coaxial:SMA_Amphenol_132289_EdgeMount
- J2: footprint (none) -> Connector_JST:JST_PH_B6B-PH-K_1x06_P2.00mm_Vertical
- L10, L11, L12, L13, L14, L15, L16, L17, L18, L19, L20, L21, L22, L23, L24, L25, L26, L27, L28, L29, L30, L7, L8, L9: footprint (none) -> Inductor_SMD:L_0402_1005Metric
- L6: footprint XFL4020-222ME -> XFL4020-222:XFL4020-222ME
- PS1: footprint QFN50P300X300X100-17N-D -> TPS62150:QFN50P300X300X100-17N-D
- Q1: footprint Package_TO_SOT_THT:TO-220-3_Horizontal_TabDown -> Package_TO_SOT_SMD:TO-252-2
- R1, R10, R11, R12, R13, R14, R15, R16, R17, R19, R2, R20, R21, R22, R23, R24, R25, R28, R29, R3, R31, R32, R33, R34, R35, R36, R37, R38, R4, R44, R45, R46, R47, R49, R5, R6, R7, R8, R9: footprint (none) -> Resistor_SMD:R_0603_1608Metric
- R39, R40, R41, R42, R43: footprint (none) -> Resistor_SMD:R_0402_1005Metric
- SW1: footprint (none) -> Button_Switch_SMD:SW_SPST_CK_KXT3
- T1, T2, T3, T4: footprint TCM163AX2 -> Balun:TCM163AX2
- Y1: footprint SiT9121AI2B133E100000000G -> REF_CLOCKS:SiT9121AI2B133E100000000G
Connections:
- net +12V: no longer C31.1, IC5.1 (IN_1), IC5.2 (IN_2), IC5.3 (EN/UV), Q1.1 (C), R29.1
- net +3.3V: now also C116.1, C117.1, D4.2 (A), R56.2; no longer C105.1, IC11.4 (VCC), R46.1
- net 5V_CLEAN: now also R62.2; no longer C44.2, C50.1, IC5.9 (OUTS), Q1.3 (E), R21.2, R24.1
- net GND: now also C109.2, C110.1, C112.2, C113.2, C114.1, C115.2, C116.2, C117.2, C119.2, C120.1, C122.2, C123.2, D1.2 (A2), IC12.11 (GND_2), IC12.5 (ILIM), IC12.8 (GND_1), IC14.11 (GND_2), IC14.5 (ILIM), IC14.8 (GND_1), PS2.15 (PGND_1), PS2.16 (PGND_2), PS2.17 (THERMAL_PAD), PS2.6 (AGND), PS2.8 (DEF), R51.2, R53.2, R54.1, R57.2, R59.2, R61.2
- net at C51.1, HMC476MP86(FREQUENZBEREICH)(nichtkomplettnotwendig)1.3 (RF-OUT_AND_DC-IN): now also L5.P$1 (RF)
- net at C46.2, C49.2, C53.2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: now also L5.P$3 (DC)
- net at C58.1, IC6.4 (RF-OUT_&_VD): now also L4.P$1 (RF)
- net BAT+: now reaches C108.1
- net BAT+: now also C31.1, C52.1, IC5.1 (IN_1), IC5.2 (IN_2), IC5.3 (EN/UV), PS1.10 (AVIN), PS1.11 (PVIN_1), PS1.12 (PVIN_2), PS1.13 (EN), Q1.1 (C), C109.1, C119.1, D1.1 (A1), D5.1 (K), IC12.1 (IN_1), IC12.2 (IN_2), IC12.3 (EN/UV), IC14.1 (IN_1), IC14.2 (IN_2), IC14.3 (EN/UV), PS2.10 (AVIN), PS2.11 (PVIN_1), PS2.12 (PVIN_2), PS2.13 (EN), Q2.1 (C), Q4.1 (C)
- net at J4.2 (Pin_2): now also SW2.2
- net at C60.1, IC7.4 (RF-OUT_&_VD): now also L2.P$1 (RF)
- net at C56.2, R30.1: now also L2.P$3 (DC)
- net at C55.2, R27.1: now also L4.P$3 (DC)
- new net: D4.1 (K), R57.1
- new net: C121.2, C123.1, IC14.9 (OUTS), Q4.3 (E), R58.2, R60.1, R64.1
- new net: C44.2, C50.1, IC5.9 (OUTS), Q1.3 (E), R21.2, R24.1, R62.1
- new net: C122.1, IC14.7 (SET), R59.1
- new net: D5.2 (A), SW2.1
- new net: C120.2, C121.1, IC14.10 (OUT), Q4.2 (B), R58.1
- new net: IC14.6 (PGFB), R60.2, R61.1
- new net: C110.2, C111.1, IC12.10 (OUT), Q2.2 (B), R50.1
- new net: C111.2, C113.1, IC12.9 (OUTS), Q2.3 (E), R50.2, R52.1, R63.1
- new net: L31.1, PS2.1 (SW_1), PS2.2 (SW_2), PS2.3 (SW_3)
- new net: C115.1, L31.2, PS2.14 (VOS), PS2.7 (FSW), R55.2, R56.1
- new net: PS2.5 (FB), R54.2, R55.1
- new net: IC12.6 (PGFB), R52.2, R53.1
- new net: C112.1, IC12.7 (SET), R51.1
- new net: C114.2, PS2.9 (SS/TR)
- new net 12V_CLEAN: R29.1, R63.2
- new net VCC_ADC: C105.1, IC11.4 (VCC), R46.1, R64.2
Other:
- moved on the sheet: C31, C42, C44, C45, C50, C52, C54, C60, C67, C76, C80, D3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

Commit message: layout
Connections:
- net +12V is gone; now on net 12V_CLEAN: R23.1
- net at IC9.10 (LOIN): now also C72.1; no longer C73.1
- net at IC9.9 (LOIP): now also C73.1; no longer C72.1
- net at IC10.10 (LOIN): now also C77.1; no longer C78.1
- net at IC10.9 (LOIP): now also C78.1; no longer C77.1
Changed lines of the file:
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@@
 	(wire
 		(pts
+			(xy 570.23 419.1) (xy 570.23 433.07)
+		)
+		(stroke
+			(width 0)
+			(type default)
+		)
+	)
+	(wire
+		(pts
 			(xy 287.02 85.09) (xy 293.37 85.09)
 		)
@@
 	(wire
 		(pts
-			(xy 567.69 433.07) (xy 576.58 433.07)
-		)
-		(stroke
-			(width 0)
-			(type default)
-		)
-	)
-	(wire
-		(pts
 			(xy 623.57 275.59) (xy 626.11 275.59)
 		)
@@
 	(wire
 		(pts
+			(xy 562.61 300.99) (xy 562.61 314.96)
+		)
+		(stroke
+			(width 0)
+			(type default)
+		)
+	)
+	(wire
+		(pts
 			(xy 83.82 281.94) (xy 86.36 281.94)
 		)
@@
 	(wire
 		(pts
+			(xy 560.07 320.04) (xy 568.96 320.04)
+		)
+		(stroke
+			(width 0)
+			(type default)
+		)
+	)
+	(wire
+		(pts
+			(xy 567.69 438.15) (xy 576.58 438.15)
+		)
+		(stroke
+			(width 0)
+			(type default)
+		)
+	)
+	(wire
+		(pts
 			(xy 544.83 270.51) (xy 544.83 273.05)
 		)
@@
 	(wire
 		(pts
+			(xy 567.69 419.1) (xy 567.69 438.15)
+		)
+		(stroke
+			(width 0)
+			(type default)
+		)
+	)
+	(wire
+		(pts
 			(xy 638.81 382.27) (xy 641.35 382.27)
 		)
@@
 	(wire
 		(pts
-			(xy 560.07 300.99) (xy 560.07 314.96)
+			(xy 560.07 300.99) (xy 560.07 320.04)
 		)
 		(stroke
@@
 	(wire
 		(pts
+			(xy 562.61 314.96) (xy 568.96 314.96)
+		)
+		(stroke
+			(width 0)
+			(type default)
+		)
+	)
+	(wire
+		(pts
 			(xy 167.64 228.6) (xy 167.64 233.68)
 		)
@@
 	(wire
 		(pts
+			(xy 570.23 433.07) (xy 576.58 433.07)
+		)
+		(stroke
+			(width 0)
+			(type default)
+		)
+	)
+	(wire
+		(pts
 			(xy 347.98 487.68) (xy 300.99 487.68)
 		)
@@
 	(wire
 		(pts
-			(xy 560.07 314.96) (xy 568.96 314.96)
-		)
-		(stroke
-			(width 0)
-			(type default)
-		)
-	)
-	(wire
-		(pts
 			(xy 59.69 265.43) (xy 59.69 270.51)
 		)
@@
 	(wire
 		(pts
-			(xy 562.61 300.99) (xy 562.61 320.04)
-		)
-		(stroke
-			(width 0)
-			(type default)
-		)
-	)
-	(wire
-		(pts
 			(xy 513.08 396.24) (xy 516.89 396.24)
 		)
@@
 	(wire
 		(pts
-			(xy 570.23 419.1) (xy 570.23 438.15)
-		)
-		(stroke
-			(width 0)
-			(type default)
-		)
-	)
-	(wire
-		(pts
 			(xy 114.3 204.47) (xy 114.3 205.74)
 		)
@@
 	(wire
 		(pts
-			(xy 568.96 320.04) (xy 562.61 320.04)
-		)
-		(stroke
-			(width 0)
-			(type default)
-		)
-	)
-	(wire
-		(pts
 			(xy 619.76 396.24) (xy 619.76 407.67)
 		)
@@
 	(wire
 		(pts
-			(xy 576.58 438.15) (xy 570.23 438.15)
-		)
-		(stroke
-			(width 0)
-			(type default)
-		)
-	)
-	(wire
-		(pts
 			(xy 284.48 100.33) (xy 287.02 100.33)
 		)
@@
 	(wire
 		(pts
-			(xy 567.69 419.1) (xy 567.69 433.07)
-		)
-		(stroke
-			(width 0)
-			(type default)
-		)
-	)
-	(wire
-		(pts
 			(xy 586.74 543.56) (xy 586.74 546.1)
 		)
@@
 		)
 	)
+	(global_label "12V_CLEAN"
+		(shape input)
+		(at 433.07 92.71 180)
+		(fields_autoplaced yes)
+		(effects
+			(font
+				(size 1.27 1.27)
+			)
+			(justify right)
+		)
+		(property "Intersheetrefs" "${INTERSHEET_REFS}"
+			(at 419.7434 92.71 0)
+			(effects
+				(font
+					(size 1.27 1.27)
+				)
+				(justify right)
+				(hide yes)
+			)
+		)
+	)
 	(global_label "VCC_CP"
 		(shape input)
@@
 					(unit 1)
 				)
-			)
-		)
-	)
-	(symbol
-		(lib_id "power:+12V")
-		(at 433.07 92.71 90)
-		(unit 1)
-		(exclude_from_sim no)
-		(in_bom yes)
-		(on_board yes)
-		(dnp no)
-		(fields_autoplaced yes)
-		(property "Reference" "#PWR0101"
-			(at 436.88 92.71 0)
-			(effects
-				(font
-					(size 1.27 1.27)
-				)
-				(hide yes)
-			)
-		)
-		(property "Value" "+12V"
-			(at 429.26 92.7099 90)
-			(effects
-				(font
-					(size 1.27 1.27)
-				)
-				(justify left)
-			)
-		)
-		(property "Footprint" ""
-			(at 433.07 92.71 0)
-			(effects
-				(font
-					(size 1.27 1.27)
-				)
-				(hide yes)
-			)
-		)
-		(property "Datasheet" ""
-			(at 433.07 92.71 0)
-			(effects
-				(font
-					(size 1.27 1.27)
-				)
-				(hide yes)
-			)
-		)
-		(property "Description" "Power symbol creates a global label with name \"+12V\""
-			(at 433.07 92.71 0)
-			(effects
-				(font
-					(size 1.27 1.27)
-				)
-				(hide yes)
-			)
-		)
-		(pin "1"
-		)
-		(instances
-			(project "MIMO_SAR_RADAR"
-				(path "/972558b7-3033-4797-8bf9-1b0bbeb52199"
-					(reference "#PWR0101")
-					(unit 1)
-				)

Commit message: update
Parts:
- removed C1: 2.2uF, Capacitor_SMD:C_0603_1608Metric, symbol Device:C_Small
- removed C2: 100nF, Capacitor_SMD:C_0603_1608Metric, symbol Device:C_Small
- removed TDK_HHM2952A1/auf_PCB1: DC4759J5020AHF-2, RF_Converter:Anaren_0805_2012Metric-6, symbol RF:DC4759J5020AHF-2
- added C118, C124, C125, C126, C127, C128, C129, C130, C131, C132, C133, C134, C135, C136, C25, C43, C9: 100nF, Capacitor_SMD:C_0603_1608Metric, symbol Device:C_Small
- added U4: HHM2952A1, TDK:HHM2952A1, symbol TDK:HHM2952A1
- C38, C6, C8: footprint Capacitor_SMD:C_0805_2012Metric -> Capacitor_SMD:C_0603_1608Metric
Connections:
- net +3.3V: now also C118.1, C124.1, C125.1, C126.1, C127.1, C128.1, C129.1, C130.1, C131.1, C132.1, C133.1, C134.1, C135.1, C136.1, C25.1, C43.1, C9.1
- net GND: now also C118.2, C124.2, C125.2, C126.2, C127.2, C128.2, C129.2, C130.2, C131.2, C132.2, C133.2, C134.2, C135.2, C136.2, C25.2, C43.2, C9.2, U4.4 (Direct), U4.5 (GND)
- net SPLIT_TX: now also U4.1 (Coupled)
- net VCC_VCO: no longer C76.1, C80.1, D3.2 (A)
- net at R39.1: now also U4.3 (Isolated)
- net at C67.1, L6.2, PS1.14 (VOS)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: now also C76.1, C80.1, D3.2 (A)
- net at FL6.3 (OUTPUT): now also U4.6 (Input)
- net at J8.1 (In): now also U4.4 (Direct)
Other:
- moved on the sheet: R35
