File: MIMO_SAR_RADAR.kicad_pcb (KiCad board)
At the start: 2 copper layers, 50 parts, among them IC1 SKY13418-485LF, IC10 PSA2-6+, IC11 ADL5380ACPZ-R7, IC12 PSA2-6+, IC13 ADL5380ACPZ-R7, IC14 OPA1632DGNR, IC15 SKY13418-485LF, IC2 AD7380-4BCPZ, IC2 SKY13418-485LF, IC21 LMX2594RHAT, IC22 SKY13418-485LF, IC23 SKY13418-485LF, IC3 ADS8584SIPM, IC4 OPA1632DGNR, IC5 LT3042IMSE#PBF, IC6 PMA3-73-1W+, IC7 OPA1632DGNR, IC8 SKY13418-485LF, IC9 OPA1632DGNR, J3 Conn_Coaxial_Small, J4 Conn_01x02_Pin, Q1 D44VH10, T1 TCM1-63AX-2+, T2 TCM1-63AX-2+, T3 TCM1-63AX-2+, T4 TCM1-63AX-2+, U1 LM2596S-12, U2 STM32H7A3IGTx, U3 ESP32-C3-WROOM-02, U5 LM1117DT-3.3, Y1 SiT9121AI-2B1-33E100.000000G

Commit message: finishing up schematic
Parts:
- removed C13: 100pF, Capacitor_SMD:C_0402_1005Metric
- removed C16, C74: 0.1uF, Capacitor_SMD:C_0603_1608Metric
- removed C73: 0.01uF, Capacitor_SMD:C_0603_1608Metric
- removed FL10, FL7, FL8: HFCG-3000+, RF_HP:HFCG3000
- removed FL9: LFCN-6000+, RF_LP:LFCN6000
- removed HMC476MP86(FREQUENZBEREICH)1: ERA-3+, ERA-3+:ERA3
- removed IC12: PSA2-6+, LNA:SOT65P215X100-6N
- removed IC13: ADL5380ACPZ-R7, RF_Modulators:QFN50P400X400X100-25N
- removed IC14: OPA1632DGNR, DIFF_AMPS:SOP65P490X110-9N
- removed IC15, IC22, IC23: SKY13418-485LF, SKY13:SKY13418485LF
- removed the IC2 at (49.4, 81.6)
- removed the IC2 at (119.1, 68.2)
- removed IC21: LMX2594RHAT, LMX:QFN50P600X600X100-41N-D
- removed PS2: LM27762DSSR, LM27762DSSR:SON50P200X300X80-13N-D
- removed R6, R9: 93.1R, Resistor_SMD:R_0805_2012Metric
- removed U5: LM1117DT-3.3, Package_TO_SOT_SMD:TO-252-3_TabPin2
- added C41: 100pF, Capacitor_SMD:C_0402_1005Metric, F.Cu at (102.6, 74.5)
- added C5: 4.7uF, Capacitor_SMD:C_0603_1608Metric, F.Cu at (95.8, 19.6)
- added C51: 100pF, Capacitor_SMD:C_0402_1005Metric, F.Cu at (102.6, 76.5)
- added C55: 0.01uF, Capacitor_SMD:C_0603_1608Metric, F.Cu at (95.8, 24.6)
- added C56: 0.01uF, Capacitor_SMD:C_0603_1608Metric, F.Cu at (95.8, 27.1)
- added C59: 0.1uF, Capacitor_SMD:C_0603_1608Metric, F.Cu at (95.8, 32.1)
- added C6: 10uF, Capacitor_SMD:C_0805_2012Metric, F.Cu at (103.4, 69.0)
- added C7: 220pF, Capacitor_SMD:C_0603_1608Metric, F.Cu at (95.8, 22.1)
- added FL3: HFCG-3000+, RF_HP:HFCG3000, F.Cu at (49.9, 77.4)
- added FL4: HFCG-3000+, RF_HP:HFCG3000, F.Cu at (55.0, 77.4)
- added FL5: LFCN-6000+, RF_LP:LFCN6000, F.Cu at (87.2, 83.0)
- added FL6: HFCG-3000+, RF_HP:HFCG3000, F.Cu at (60.1, 77.4)
- added HMC476MP86(FREQUENZBEREICH)(nichtkomplettnotwendig)1: ERA-3+, ERA-3+:ERA3, F.Cu at (96.1, 72.7)
- added IC2: SKY13418-485LF, SKY13:SKY13418485LF, F.Cu at (55.5, 71.7)
- added J10: Conn_01x06_Pin, Connector_JST:JST_PH_B6B-PH-K_1x06_P2.00mm_Vertical, F.Cu at (106.2, 51.5)
- added J5: Conn_Coaxial_Small, Connector_Coaxial:SMA_Amphenol_132289_EdgeMount, F.Cu at (68.5, 51.0)
- added J6: Conn_Coaxial_Small, Connector_Coaxial:SMA_Amphenol_132289_EdgeMount, F.Cu at (68.5, 63.2)
- added J7: Conn_01x06_Pin, Connector_JST:JST_PH_B6B-PH-K_1x06_P2.00mm_Vertical, F.Cu at (106.5, 39.8)
- added J8: Conn_Coaxial_Small, Connector_Coaxial:SMA_Amphenol_132289_EdgeMount, F.Cu at (68.5, 75.4)
- added J9: Conn_01x06_Pin, Connector_JST:JST_PH_B6B-PH-K_1x06_P2.00mm_Vertical, F.Cu at (106.2, 45.5)
- added L6: XFL4020-222MEB, XFL4020-222:XFL4020-222ME, F.Cu at (74.9, 84.1)
- added R27: 93.1R, Resistor_SMD:R_0805_2012Metric, F.Cu at (103.3, 58.7)
- added R30: 93.1R, Resistor_SMD:R_0805_2012Metric, F.Cu at (103.3, 61.7)
- added U4: LM1117DT-3.3, Package_TO_SOT_SMD:TO-252-3_TabPin2, F.Cu at (97.8, 82.0)
- C57: value 0.01uF -> 0.1uF
- C8: value 100pF -> 10uF; footprint Capacitor_SMD:C_0402_1005Metric -> Capacitor_SMD:C_0805_2012Metric
- IC10: value PSA2-6+ -> ADL5380ACPZ-R7; footprint LNA:SOT65P215X100-6N -> RF_Modulators:QFN50P400X400X100-25N
- IC11: value ADL5380ACPZ-R7 -> AD7380-4BCPZ; footprint RF_Modulators:QFN50P400X400X100-25N -> AD7380:QFN50P400X400X60-25N-D
- IC3: value ADS8584SIPM -> SKY13418-485LF; footprint 4CH_ADC:QFP50P1200X1200X160-64N -> SKY13:SKY13418485LF
- IC4: value OPA1632DGNR -> LMX2594RHAT; footprint DIFF_AMPS:SOP65P490X110-9N -> LMX:QFN50P600X600X100-41N-D
- IC6: value PMA3-73-1W+ -> PSA2-6+; footprint PMA3:QFN51P300X300X89-13N -> LNA:SOT65P215X100-6N
- IC7: value OPA1632DGNR -> PSA2-6+; footprint DIFF_AMPS:SOP65P490X110-9N -> LNA:SOT65P215X100-6N
- IC8: value SKY13418-485LF -> PMA3-73-1W+; footprint SKY13:SKY13418485LF -> PMA3:QFN51P300X300X89-13N
- IC9: value OPA1632DGNR -> ADL5380ACPZ-R7; footprint DIFF_AMPS:SOP65P490X110-9N -> RF_Modulators:QFN50P400X400X100-25N
- J3: value Conn_Coaxial_Small -> SWD; footprint Connector_Coaxial:SMA_Amphenol_132289_EdgeMount -> Connector_JST:JST_XH_B4B-XH-A_1x04_P2.50mm_Vertical
- L1: value XFL4020-222MEB -> 2.2uH; footprint XFL4020-222:XFL4020-222ME -> Inductor_SMD:L_0805_2012Metric_Pad1.15x1.40mm_HandSolder
- U1: value LM2596S-12 -> STM32H745IITx; footprint Package_TO_SOT_SMD:TO-263-5_TabPin3 -> Package_QFP:LQFP-176_24x24mm_P0.5mm
- U2: value STM32H7A3IGTx -> ESP32-C3-WROOM-02; footprint Package_QFP:LQFP-176_24x24mm_P0.5mm -> RF_Module:ESP32-C3-WROOM-02
- U3: value ESP32-C3-WROOM-02 -> LM2596S-12; footprint RF_Module:ESP32-C3-WROOM-02 -> Package_TO_SOT_SMD:TO-263-5_TabPin3
- moved IC8 88.1 mm to (38.5, 79.3)
- moved Y1 70.9 mm to (50.6, 83.2)
- moved Q1 69.4 mm to (39.1, 74.9)
- moved IC7 69.3 mm to (43.4, 82.4)
- moved FL2 62.5 mm to (87.2, 76.8)
- moved T3 62.0 mm to (53.1, 50.7)
- moved T4 62.0 mm to (60.0, 50.7)
- moved PS1 61.5 mm to (38.5, 84.6)
- moved T2 59.8 mm to (46.2, 50.7)
- moved T1 59.8 mm to (39.3, 50.7)
- moved IC6 57.6 mm to (43.4, 78.6)
- moved J3 56.2 mm to (50.9, 64.6)
- moved IC5 49.8 mm to (68.0, 83.9)
- moved U1 47.3 mm to (50.0, 32.5)
- moved FL1 45.4 mm to (87.2, 70.6)
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Connections:
- net RX1_B0 renamed Net-(IC1-V1)
- net RX1_B1 renamed Net-(IC1-V2)
- C57 pad 1: GND -> VSS
- C57 pad 2: Net-(C57-Pad2) -> 5V_CLEAN
- C8 pad 1: Net-(IC21-RFOUTAP) -> VCAP
- C8 pad 2: Net-(HMC476MP86(FREQUENZBEREICH)1-RF_IN) -> VSS
- FL1 pad 2: GND -> VSS
- FL1 pad 4: GND -> VSS
- FL2 pad 2: GND -> VSS
- FL2 pad 4: GND -> VSS
- IC1 pad 13: Net-(FL1-RF_IN) -> Net-(IC1-ANT)
- IC1 pad 15: GND -> VSS
- IC1 pad 3: unconnected-(IC1-RF1-Pad3) -> Net-(IC1-RF1)
- IC1 pad 4: +3.3V -> VDDSMPS
- IC1 pad 5: RX1_B2 -> RF_SWITCH_BIT_0
- IC1 pad 9: unconnected-(IC1-RF2-Pad9) -> Net-(IC1-RF2)
- IC10 pad 1: Net-(IC10-RF-IN) -> VSS
- IC10 pad 2: GND -> VSS
- IC10 pad 3: GND -> IHI2
- IC10 pad 4: Net-(IC10-RF-OUT_&_VD) -> ILO2
- IC10 pad 5: GND -> VSS
- IC10 pad 6: GND -> 5V_CLEAN
- IC11 pad 1: GND -> VSS
- IC11 pad 10: Net-(IC11-LOIN) -> ADC_B-
- IC11 pad 11: GND -> ADC_B+
- IC11 pad 12: unconnected-(IC11-NC-Pad12) -> ADC_A-
- IC11 pad 13: 5V_CLEAN -> ADC_A+
- IC11 pad 14: GND -> VSS
- IC11 pad 15: Net-(IC11-QLO) -> unconnected-(IC11-DNC-Pad15)
- IC11 pad 16: Net-(IC11-QHI) -> VSS
- IC11 pad 17: GND -> Net-(IC11-REFIO)
- IC11 pad 18: GND -> CSNOT
- IC11 pad 19: Net-(IC11-ADJ) -> SDOA
- IC11 pad 2: GND -> VCC
- IC11 pad 20: GND -> SDOB
- IC11 pad 21: Net-(IC11-REFIN) -> SDI_ADC
- IC11 pad 22: Net-(IC11-REFIP) -> SCLK_ADC
- IC11 pad 23: GND -> SDOC
- IC11 pad 24: 5V_CLEAN -> SDOD
- IC11 pad 25: unconnected-(IC11-EP-Pad25) -> VSS
- IC11 pad 3: IHI1 -> Net-(IC11-REGCAP)
- IC11 pad 4: ILO1 -> VDDSMPS
- IC11 pad 5: GND -> VSS
- IC11 pad 6: 5V_CLEAN -> ADC_D-
- IC11 pad 7: Net-(IC11-ENBL) -> ADC_D+
- IC11 pad 8: GND -> ADC_C-
- IC11 pad 9: Net-(IC11-LOIP) -> ADC_C+
- IC3 pad 13: unconnected-(IC3-~{CS}-Pad13) -> Net-(IC1-RF1)
- IC3 pad 15: unconnected-(IC3-FRSTDATA-Pad15) -> VSS
- IC3 pad 4: unconnected-(IC3-OS1-Pad4) -> VDDSMPS
- IC3 pad 5: unconnected-(IC3-OS2-Pad5) -> RF_SWITCH_BIT_3
- IC3 pad 6: unconnected-(IC3-~{PAR}/SER/BYTE_SEL-Pad6) -> RF_SWITCH_BIT_2
- IC3 pad 7: unconnected-(IC3-~{STBY}-Pad7) -> RF_SWITCH_BIT_1
- IC4 pad 2: GND -> VSS
- IC4 pad 3: unconnected-(IC4-V+-Pad3) -> Net-(IC4-VBIASVCO)
- IC4 pad 4: unconnected-(IC4-VOUT+-Pad4) -> VSS
- IC4 pad 5: unconnected-(IC4-VOUT--Pad5) -> Net-(IC4-SYNC)
- IC4 pad 6: unconnected-(IC4-V--Pad6) -> VSS
- IC4 pad 7: Net-(IC4-ENABLE) -> VCC_DIG
- IC4 pad 8: Net-(IC4-VIN+) -> OSC_IN_P_FILTERED
- IC4 pad 9: GND -> OSC_IN_M_FILTERED
- IC5 pad 11: GND -> VSS
- IC5 pad 5: GND -> VSS
- IC5 pad 8: GND -> VSS
- IC6 pad 1: GND -> Net-(IC6-RF-IN)
- IC6 pad 2: Net-(IC6-RF-IN) -> VSS
- IC6 pad 3: GND -> VSS
- IC6 pad 4: unconnected-(IC6-NC_1-Pad4) -> Net-(IC6-RF-OUT_&_VD)
- IC6 pad 5: unconnected-(IC6-NC_2-Pad5) -> VSS
- IC6 pad 6: unconnected-(IC6-NC_3-Pad6) -> VSS
- IC7 pad 2: GND -> VSS
- IC7 pad 3: unconnected-(IC7-V+-Pad3) -> VSS
- IC7 pad 4: unconnected-(IC7-VOUT+-Pad4) -> Net-(IC7-RF-OUT_&_VD)
- IC7 pad 5: unconnected-(IC7-VOUT--Pad5) -> VSS
- IC7 pad 6: unconnected-(IC7-V--Pad6) -> VSS
- IC8 pad 1: unconnected-(IC8-RF5-Pad1) -> VSS
- IC8 pad 12: unconnected-(IC8-RF8-Pad12) -> Net-(IC8-VIADJ)
- IC8 pad 13: Net-(FL2-RF_IN) -> VSS
- IC8 pad 2: unconnected-(IC8-RF3-Pad2) -> Net-(IC8-RF-IN)
- IC8 pad 3: unconnected-(IC8-RF1-Pad3) -> VSS
- IC8 pad 4: +3.3V -> unconnected-(IC8-NC_1-Pad4)
- IC8 pad 7: unconnected-(IC8-V1-Pad7) -> VSS
- IC8 pad 8: unconnected-(IC8-N/C-Pad8) -> Net-(FL5-RF_IN)
- IC8 pad 9: unconnected-(IC8-RF2-Pad9) -> VSS
- IC9 pad 1: Net-(IC9-VIN-) -> VSS
- IC9 pad 2: GND -> VSS
- IC9 pad 3: unconnected-(IC9-V+-Pad3) -> IHI1
- IC9 pad 4: unconnected-(IC9-VOUT+-Pad4) -> ILO1
- IC9 pad 5: unconnected-(IC9-VOUT--Pad5) -> VSS
- IC9 pad 6: unconnected-(IC9-V--Pad6) -> 5V_CLEAN
- IC9 pad 8: Net-(IC9-VIN+) -> VSS
- IC9 pad 9: GND -> Net-(IC9-LOIP)
- J3 pad 1: Net-(J3-In) -> VDDSMPS
- J3 pad 2: GND -> SWCLK
- J4 pad 1: GND -> VSS
- L1 pad 1: Net-(PS1-SW_1) -> VCAP
- L1 pad 2: Net-(PS1-FSW) -> VLXSMPS
- PS1 pad 15: GND -> VSS
- PS1 pad 16: GND -> VSS
- PS1 pad 17: GND -> VSS
- PS1 pad 6: GND -> VSS
- PS1 pad 8: GND -> VSS
- T1 pad 2: GND -> VSS
- T1 pad 3: SPLIT_TX -> RX1_BALUN_IN
- T2 pad 2: GND -> VSS
- T2 pad 3: RX1_BALUN_IN -> SPLIT_TX
- T3 pad 2: GND -> VSS
- T4 pad 2: GND -> VSS
- TDK_HHM2952A1/auf_PCB1 pad 3: GND -> VSS
- TDK_HHM2952A1/auf_PCB1 pad 4: GND -> VSS
- TDK_HHM2952A1/auf_PCB1 pad 6: Net-(J3-In) -> Net-(J8-In)
- U1 pad 1: Net-(D3-K) -> unconnected-(U1-PE2-Pad1)
- U1 pad 2: Net-(D2-K) -> unconnected-(U1-PE3-Pad2)
- U1 pad 3: GND -> unconnected-(U1-PE4-Pad3)
- U1 pad 4: Net-(U1-FB) -> unconnected-(U1-PE5-Pad4)
- U1 pad 5: GND -> unconnected-(U1-PE6-Pad5)
- U2 pad 14: GND -> unconnected-(U2-IO19-Pad14)
- U2 pad 15: +3.3V -> unconnected-(U2-IO3-Pad15)
- U2 pad 19: unconnected-(U2-PF3-Pad19) -> VSS
- U2 pad 9: unconnected-(U2-PC14-Pad9) -> VSS
- U3 pad 1: unconnected-(U3-3V3-Pad1) -> Net-(D1-K)
- U3 pad 2: unconnected-(U3-EN-Pad2) -> Net-(D2-K)
- U3 pad 3: unconnected-(U3-IO4-Pad3) -> VSS
- U3 pad 4: unconnected-(U3-IO5-Pad4) -> Net-(U3-FB)
- U3 pad 5: unconnected-(U3-IO6-Pad5) -> VSS
- Y1 pad 3: GND -> VSS
- Y1 pad 6: +3.3V -> VDDSMPS

Commit message: battery system angefangen
Parts:
- added BT1: Battery_Cell, Battery:BatteryHolder_Keystone_1042_1x18650, F.Cu at (168.0, 57.2)
- added BT1: Battery_Cell, Battery:BatteryHolder_Keystone_1042_1x18650, F.Cu at (190.0, 56.8)
- added BT1: Battery_Cell, Battery:BatteryHolder_Keystone_1042_1x18650, F.Cu at (212.5, 57.0)
- added C43: 680uF, Capacitor_SMD:C_Elec_10x10.2, F.Cu at (146.4, 59.0)
- added C9: 680uF, Capacitor_SMD:C_Elec_10x10.2, F.Cu at (129.6, 55.8)
- added U5: LM2596S-3.3, Package_TO_SOT_SMD:TO-263-5_TabPin3, F.Cu at (132.8, 43.6)
- moved Q1 98.8 mm to (119.6, 17.7), turned to -90 degrees
- moved J8 50.5 mm to (30.4, 42.3), turned to 180 degrees
- moved U3 43.2 mm to (132.9, 31.8)
- moved J5 41.3 mm to (30.4, 66.7), turned to 180 degrees
- moved U4 39.5 mm to (134.9, 68.3)
- moved J6 39.1 mm to (30.4, 54.5), turned to 180 degrees
- moved J4 27.7 mm to (115.8, 68.2)
- moved U2 2.26 mm to (77.7, 35.4)
Connections:
- U1 pad 150: unconnected-(U1-PD7-Pad150) -> Net-(U1-PD7)
- U2 pad 1: unconnected-(U2-3V3-Pad1) -> VDDSMPS
- U2 pad 16: unconnected-(U2-IO2-Pad16) -> Net-(U1-PD7)
- U2 pad 2: unconnected-(U2-EN-Pad2) -> Net-(U2-EN)

Commit message: layout
Parts:
- removed BT1 (x3): Battery_Cell, Battery:BatteryHolder_Keystone_1042_1x18650
- removed C43, C9: 680uF, Capacitor_SMD:C_Elec_10x10.2
- removed U3: LM2596S-12, Package_TO_SOT_SMD:TO-263-5_TabPin3
- removed U4: LM1117DT-3.3, Package_TO_SOT_SMD:TO-252-3_TabPin2
- removed U5: LM2596S-3.3, Package_TO_SOT_SMD:TO-263-5_TabPin3
- added C1: 2.2uF, Capacitor_SMD:C_0603_1608Metric, F.Cu at (94.0, 116.6)
- added C10: 0.1uF, Capacitor_SMD:C_0402_1005Metric, F.Cu at (134.0, 115.8)
- added C100: C_Small, Capacitor_SMD:C_0402_1005Metric, F.Cu at (163.7, 107.5)
- added C101: C_Small, Capacitor_SMD:C_0402_1005Metric, F.Cu at (170.6, 109.9)
- added C102: C_Small, Capacitor_SMD:C_0402_1005Metric, F.Cu at (164.6, 91.7)
- added C103: C_Small, Capacitor_SMD:C_0402_1005Metric, F.Cu at (170.0, 91.5)
- added C104: 1uF, Capacitor_SMD:C_0603_1608Metric, F.Cu at (160.1, 95.2)
- added C105: 1uF, Capacitor_SMD:C_0603_1608Metric, F.Cu at (151.2, 98.2)
- added C106: C_Small, Capacitor_SMD:C_0603_1608Metric, F.Cu at (155.2, 93.5)
- added C107: 1uF, Capacitor_SMD:C_0603_1608Metric, F.Cu at (157.9, 96.2)
- added C108: 10uF, Capacitor_SMD:C_0603_1608Metric, F.Cu at (70.8, 77.8)
- added C109: 4.7uF, Capacitor_SMD:C_0603_1608Metric, F.Cu at (68.5, 104.5)
- added C11: 0.1uF, Capacitor_SMD:C_0402_1005Metric, F.Cu at (133.6, 111.5)
- added C110: C_Small, Capacitor_SMD:C_0603_1608Metric, F.Cu at (60.2, 98.6)
- added C111: 10uF, Capacitor_SMD:C_0603_1608Metric, F.Cu at (67.4, 93.4)
- added C112: 0.47pF, Capacitor_SMD:C_0603_1608Metric, F.Cu at (62.0, 93.5)
- added C113: 10uF, Capacitor_SMD:C_0603_1608Metric, F.Cu at (63.8, 93.6)
- added C114: 3.3nF, Capacitor_SMD:C_0603_1608Metric, F.Cu at (66.3, 74.2)
- added C115: 22uF, Capacitor_SMD:C_0805_2012Metric, F.Cu at (75.8, 69.0)
- added C116: 0.1uF, Capacitor_SMD:C_0603_1608Metric, F.Cu at (68.5, 65.5)
- added C117: 10uF, Capacitor_SMD:C_0603_1608Metric, F.Cu at (73.2, 65.5)
- added C119: 4.7uF, Capacitor_SMD:C_0603_1608Metric, F.Cu at (69.2, 89.5)
- added C12: 0.1uF, Capacitor_SMD:C_0603_1608Metric, F.Cu at (131.3, 110.6)
- added C120: C_Small, Capacitor_SMD:C_0603_1608Metric, F.Cu at (60.4, 83.4)
- added C121: 10uF, Capacitor_SMD:C_0603_1608Metric, F.Cu at (68.2, 78.6)
- added C122: 0.47pF, Capacitor_SMD:C_0603_1608Metric, F.Cu at (62.8, 78.6)
- added C123: 10uF, Capacitor_SMD:C_0603_1608Metric, F.Cu at (64.6, 78.6)
- added C13: 0.1uF, Capacitor_SMD:C_0603_1608Metric, F.Cu at (134.0, 124.3)
- added C14: 0.1uF, Capacitor_SMD:C_0603_1608Metric, F.Cu at (131.4, 126.8)
- added C15: 0.1uF, Capacitor_SMD:C_0603_1608Metric, F.Cu at (131.5, 123.3)
- added C16: 0.1uF, Capacitor_SMD:C_0603_1608Metric, F.Cu at (117.7, 122.1)
- added C17: 0.1uF, Capacitor_SMD:C_0603_1608Metric, F.Cu at (125.5, 126.7)
- added C18: 10uF, Capacitor_SMD:C_0603_1608Metric, F.Cu at (129.8, 110.6)
- added C19: 1uF, Capacitor_SMD:C_0603_1608Metric, F.Cu at (135.6, 124.3)
- added C2: 100nF, Capacitor_SMD:C_0603_1608Metric, F.Cu at (96.5, 116.6)
- added C20: 1uF, Capacitor_SMD:C_0603_1608Metric, F.Cu at (131.4, 125.2)
- added C21: 10uF, Capacitor_SMD:C_0603_1608Metric, F.Cu at (131.5, 121.8)
- added C22: 1uF, Capacitor_SMD:C_0603_1608Metric, F.Cu at (117.7, 120.5)
- added C23: 10uF, Capacitor_SMD:C_0603_1608Metric, F.Cu at (125.5, 125.1)
- added C24: 10uF (X7R), Capacitor_SMD:C_0402_1005Metric, F.Cu at (124.8, 120.9)
- added C26: 1uF, Capacitor_SMD:C_0603_1608Metric, F.Cu at (127.3, 122.5)
- added C27: C_Small, Capacitor_SMD:C_0402_1005Metric, F.Cu at (130.1, 117.2)
- added C28: C_Small, Capacitor_SMD:C_0402_1005Metric, F.Cu at (132.8, 118.1)
- added C29: 1uF, Capacitor_SMD:C_0603_1608Metric, F.Cu at (119.6, 118.1)
- added C3: 4.7uF, Capacitor_SMD:C_0603_1608Metric, F.Cu at (99.0, 116.6)
- added C30: 10uF, Capacitor_SMD:C_0603_1608Metric, F.Cu at (119.7, 116.6)
- added C31: 4.7uF, Capacitor_SMD:C_0603_1608Metric, F.Cu at (68.5, 119.8)
- added C32: C_Small, Capacitor_SMD:C_0603_1608Metric, F.Cu at (119.6, 115.1)
- added C33: 10pF Np0/C0G 0402, Capacitor_SMD:C_0402_1005Metric, F.Cu at (130.1, 114.3)
- added C34: 10pF Np0/C0G 0402, Capacitor_SMD:C_0402_1005Metric, F.Cu at (130.2, 113.0)
- added C35: 10uF, Capacitor_SMD:C_0603_1608Metric, F.Cu at (119.7, 113.6)
- added C36: 1uF, Capacitor_SMD:C_0603_1608Metric, F.Cu at (123.8, 110.6)
- added C37: 10uF, Capacitor_SMD:C_0603_1608Metric, F.Cu at (134.9, 112.1)
- added C38: 10uF, Capacitor_SMD:C_0805_2012Metric, F.Cu at (105.0, 115.8)
- added C39: 10pF Np0/C0G 0402, Capacitor_SMD:C_0402_1005Metric, F.Cu at (127.8, 110.2)
- added C4: C_Small, Capacitor_SMD:C_0603_1608Metric, F.Cu at (100.7, 114.8)
- added C40: 10uF, Capacitor_SMD:C_0603_1608Metric, F.Cu at (122.2, 110.6)
- added C42: C_Small, Capacitor_SMD:C_0603_1608Metric, F.Cu at (60.1, 113.7)
- added C44: 10uF, Capacitor_SMD:C_0603_1608Metric, F.Cu at (67.3, 108.7)
- added C45: 0.47pF, Capacitor_SMD:C_0603_1608Metric, F.Cu at (62.0, 108.6)
- added C46: 2.2uF, Capacitor_SMD:C_0603_1608Metric, F.Cu at (117.1, 96.4)
- added C47: 2400pF, Capacitor_SMD:C_0402_1005Metric, F.Cu at (192.2, 121.7)
- added C48: 2400pF, Capacitor_SMD:C_0603_1608Metric, F.Cu at (174.0, 68.4)
- added C49: 1000pF, Capacitor_SMD:C_0603_1608Metric, F.Cu at (117.2, 91.9)
- added C50: 10uF, Capacitor_SMD:C_0603_1608Metric, F.Cu at (63.7, 108.6)
- added C52: 10uF, Capacitor_SMD:C_0603_1608Metric, F.Cu at (84.4, 123.4)
- added C53: 100pF, Capacitor_SMD:C_0603_1608Metric, F.Cu at (117.0, 86.5)
- added C54: 3.3nF, Capacitor_SMD:C_0603_1608Metric, F.Cu at (84.4, 125.1)
- added C58: 2400pF, Capacitor_SMD:C_0402_1005Metric, F.Cu at (166.3, 130.1)
- added C60: 2400pF, Capacitor_SMD:C_0402_1005Metric, F.Cu at (187.7, 75.5)
- added C61: 100pF, Capacitor_SMD:C_0603_1608Metric, F.Cu at (170.4, 129.5)
- added C62: 0.1uF, Capacitor_SMD:C_0603_1608Metric, F.Cu at (168.8, 129.4)
- added C63: 100pF, Capacitor_SMD:C_0603_1608Metric, F.Cu at (171.0, 68.6)
- added C64: 0.1uF, Capacitor_SMD:C_0603_1608Metric, F.Cu at (170.9, 70.3)
- added C65: 100pF, Capacitor_SMD:C_0603_1608Metric, F.Cu at (162.6, 128.5)
- added C66: 0.1uF, Capacitor_SMD:C_0603_1608Metric, F.Cu at (164.2, 128.5)
- added C67: 22uF, Capacitor_SMD:C_0805_2012Metric, F.Cu at (80.7, 128.5)
- added C68: 100pF, Capacitor_SMD:C_0603_1608Metric, F.Cu at (173.8, 70.3)
- added C69: 0.1uF, Capacitor_SMD:C_0603_1608Metric, F.Cu at (172.2, 71.8)
- added C70: 100pF, Capacitor_SMD:C_0402_1005Metric, F.Cu at (159.2, 125.2)
- added C71: 100pF, Capacitor_SMD:C_0402_1005Metric, F.Cu at (159.3, 122.7)
- added C72: 100pF, Capacitor_SMD:C_0402_1005Metric, F.Cu at (172.5, 122.8)
- added C73: 100pF, Capacitor_SMD:C_0402_1005Metric, F.Cu at (172.4, 124.9)
- added C74: 100pF, Capacitor_SMD:C_0402_1005Metric, F.Cu at (172.5, 73.1)
- added C75: 100pF, Capacitor_SMD:C_0402_1005Metric, F.Cu at (172.5, 74.6)
- added C76: 0.1uF, Capacitor_SMD:C_0603_1608Metric, F.Cu at (81.8, 131.0)
- added C77: 100pF, Capacitor_SMD:C_0402_1005Metric, F.Cu at (162.1, 75.5)
- added C78: 100pF, Capacitor_SMD:C_0402_1005Metric, F.Cu at (161.8, 73.1)
- added C79: 0.1uF, Capacitor_SMD:C_0603_1608Metric, F.Cu at (171.2, 119.7)
- added C80: 10uF, Capacitor_SMD:C_0603_1608Metric, F.Cu at (82.6, 128.4)
- added C81: 100pF, Capacitor_SMD:C_0603_1608Metric, F.Cu at (169.6, 121.2)
- added C82: 0.1uF, Capacitor_SMD:C_0603_1608Metric, F.Cu at (170.7, 67.0)
- added C83: 100pF, Capacitor_SMD:C_0603_1608Metric, F.Cu at (166.5, 67.7)
- added C84: 10uF, Capacitor_SMD:C_0402_1005Metric, F.Cu at (162.3, 117.9)
- added C85: 10uF, Capacitor_SMD:C_0402_1005Metric, F.Cu at (165.2, 118.0)
- added C86: 10uF, Capacitor_SMD:C_0402_1005Metric, F.Cu at (168.6, 118.0)
- added C87: 10uF, Capacitor_SMD:C_0402_1005Metric, F.Cu at (172.6, 118.0)
- added C88: 10uF, Capacitor_SMD:C_0402_1005Metric, F.Cu at (166.0, 81.9)
- added C89: 10uF, Capacitor_SMD:C_0402_1005Metric, F.Cu at (162.9, 81.9)
- added C90: 10uF, Capacitor_SMD:C_0402_1005Metric, F.Cu at (171.4, 82.0)
- added C91: 10uF, Capacitor_SMD:C_0402_1005Metric, F.Cu at (168.6, 82.0)
- added C92: C_Small, Capacitor_SMD:C_0402_1005Metric, F.Cu at (164.3, 114.4)
- added C93: C_Small, Capacitor_SMD:C_0402_1005Metric, F.Cu at (170.6, 115.0)
- added C94: C_Small, Capacitor_SMD:C_0402_1005Metric, F.Cu at (164.6, 85.6)
- added C95: C_Small, Capacitor_SMD:C_0402_1005Metric, F.Cu at (169.9, 85.5)
- added C96: C_Small, Capacitor_SMD:C_0402_1005Metric, F.Cu at (163.0, 111.5)
- added C97: C_Small, Capacitor_SMD:C_0402_1005Metric, F.Cu at (170.9, 112.5)
- added C98: C_Small, Capacitor_SMD:C_0402_1005Metric, F.Cu at (164.6, 88.5)
- added C99: C_Small, Capacitor_SMD:C_0402_1005Metric, F.Cu at (170.0, 88.4)
- added D1: SMF18A, Diode_SMD:D_SMF, F.Cu at (74.8, 116.6)
- added D3: VCO_POWER_CHECK, LED_SMD:LED_0603_1608Metric, F.Cu at (85.9, 128.3)
- added D4: VCO_POWER_CHECK, LED_SMD:LED_0603_1608Metric, F.Cu at (71.0, 69.2)
- added D5: SS54, Diode_SMD:D_SMA, F.Cu at (73.2, 120.2)
- added H1: MountingHole, MountingHole:MountingHole_3.2mm_M3_DIN965_Pad, F.Cu at (60.7, 129.4)
- added H1: MountingHole, MountingHole:MountingHole_3.2mm_M3_DIN965_Pad, F.Cu at (60.8, 68.5)
- added H2: MountingHole, MountingHole:MountingHole_3.2mm_M3_DIN965_Pad, F.Cu at (202.4, 131.2)
- added H3: MountingHole, MountingHole:MountingHole_3.2mm_M3_DIN965_Pad, F.Cu at (203.9, 68.7)
- added IC12: LT3042IMSE#PBF, Low_noise_LDO:SOP50P490X110-11N, F.Cu at (64.4, 104.8)
- added IC14: LT3042IMSE#PBF, Low_noise_LDO:SOP50P490X110-11N, F.Cu at (65.0, 89.8)
- added J1: Conn_Coaxial_Small, Connector_Coaxial:SMA_Amphenol_132289_EdgeMount, F.Cu at (63.5, 171.7)
- added J2: Conn_01x06_Pin, Connector_JST:JST_PH_B6B-PH-K_1x06_P2.00mm_Vertical, F.Cu at (70.3, 180.5)
- added L10: L_Small, Inductor_SMD:L_0402_1005Metric, F.Cu at (172.7, 115.5)
- added L11: L_Small, Inductor_SMD:L_0402_1005Metric, F.Cu at (166.0, 84.2)
- added L12: L_Small, Inductor_SMD:L_0402_1005Metric, F.Cu at (162.9, 84.1)
- added L13: L_Small, Inductor_SMD:L_0402_1005Metric, F.Cu at (171.4, 84.0)
- added L14: L_Small, Inductor_SMD:L_0402_1005Metric, F.Cu at (168.6, 84.1)
- added L15: L_Small, Inductor_SMD:L_0402_1005Metric, F.Cu at (162.3, 113.1)
- added L16: L_Small, Inductor_SMD:L_0402_1005Metric, F.Cu at (165.2, 113.0)
- added L17: L_Small, Inductor_SMD:L_0402_1005Metric, F.Cu at (168.6, 113.1)
- added L18: L_Small, Inductor_SMD:L_0402_1005Metric, F.Cu at (172.7, 112.9)
- added L19: L_Small, Inductor_SMD:L_0402_1005Metric, F.Cu at (166.1, 87.1)
- added L2: TCCH-80, TCCH-80:GU1604, F.Cu at (184.1, 79.8)
- added L20: L_Small, Inductor_SMD:L_0402_1005Metric, F.Cu at (162.9, 87.1)
- added L21: L_Small, Inductor_SMD:L_0402_1005Metric, F.Cu at (171.4, 86.9)
- added L22: L_Small, Inductor_SMD:L_0402_1005Metric, F.Cu at (168.6, 87.0)
- added L23: L_Small, Inductor_SMD:L_0402_1005Metric, F.Cu at (162.3, 110.1)
- added L24: L_Small, Inductor_SMD:L_0402_1005Metric, F.Cu at (165.2, 110.0)
- added L25: L_Small, Inductor_SMD:L_0402_1005Metric, F.Cu at (168.6, 110.4)
- added L26: L_Small, Inductor_SMD:L_0402_1005Metric, F.Cu at (172.8, 110.3)
- added L27: L_Small, Inductor_SMD:L_0402_1005Metric, F.Cu at (166.1, 90.0)
- added L28: L_Small, Inductor_SMD:L_0402_1005Metric, F.Cu at (162.9, 90.0)
- added L29: L_Small, Inductor_SMD:L_0402_1005Metric, F.Cu at (171.4, 89.8)
- added L30: L_Small, Inductor_SMD:L_0402_1005Metric, F.Cu at (168.6, 89.9)
- added L31: XFL4020-222MEB, XFL4020-222:XFL4020-222ME, F.Cu at (74.8, 73.5)
- added L4: TCCH-80, TCCH-80:GU1604, F.Cu at (184.7, 125.2)
- added L5: TCCH-80, TCCH-80:GU1604, F.Cu at (121.3, 95.9)
- added L7: L_Small, Inductor_SMD:L_0402_1005Metric, F.Cu at (162.4, 115.7)
- added L8: L_Small, Inductor_SMD:L_0402_1005Metric, F.Cu at (165.2, 115.9)
- added L9: L_Small, Inductor_SMD:L_0402_1005Metric, F.Cu at (168.6, 115.5)
- added PS2: TPS62150RGTR, TPS62150:QFN50P300X300X100-17N-D, F.Cu at (70.0, 73.5)
- added Q2: DPAK, Package_TO_SOT_SMD:TO-252-2, F.Cu at (65.9, 99.0)
- added Q4: D44VH10, Package_TO_SOT_SMD:TO-252-2, F.Cu at (66.1, 84.0)
- added R1: 10k, Resistor_SMD:R_0603_1608Metric, F.Cu at (78.5, 114.9)
- added R10: 1.5R, Resistor_SMD:R_0603_1608Metric, F.Cu at (134.8, 126.7)
- added R11: 1.5R, Resistor_SMD:R_0603_1608Metric, F.Cu at (129.1, 126.0)
- added R12: 1.5R, Resistor_SMD:R_0603_1608Metric, F.Cu at (129.1, 122.6)
- added R13: 1.5R, Resistor_SMD:R_0603_1608Metric, F.Cu at (120.1, 121.3)
- added R14: 1.5R, Resistor_SMD:R_0603_1608Metric, F.Cu at (123.2, 125.9)
- added R15: 10k, Resistor_SMD:R_0603_1608Metric, F.Cu at (121.8, 121.3)
- added R16: R_Small, Resistor_SMD:R_0603_1608Metric, F.Cu at (123.5, 121.3)
- added R17: werte_siehe_PLLATINUM_SIM, Resistor_SMD:R_0603_1608Metric, F.Cu at (130.6, 115.9)
- added R19: R_Small, Resistor_SMD:R_0603_1608Metric, F.Cu at (134.8, 122.0)
- added R2: R_Small, Resistor_SMD:R_0603_1608Metric, F.Cu at (89.6, 114.8)
- added R20: R_Small, Resistor_SMD:R_0603_1608Metric, F.Cu at (130.5, 118.7)
- added R21: 10k, Resistor_SMD:R_0603_1608Metric, F.Cu at (65.5, 108.6)
- added R22: 50k, Resistor_SMD:R_0603_1608Metric, F.Cu at (60.2, 110.3)
- added R23: 240R, Resistor_SMD:R_0603_1608Metric, F.Cu at (117.2, 100.0)
- added R24: 249k, Resistor_SMD:R_0603_1608Metric, F.Cu at (60.1, 117.1)
- added R25: 49k, Resistor_SMD:R_0603_1608Metric, F.Cu at (60.1, 120.4)
- added R28: 180k, Resistor_SMD:R_0603_1608Metric, F.Cu at (77.2, 124.4)
- added R29: R_Small, Resistor_SMD:R_0603_1608Metric, F.Cu at (119.5, 90.7)
- added R3: inf, Resistor_SMD:R_0603_1608Metric, F.Cu at (83.8, 117.6)
- added R31: R_Small, Resistor_SMD:R_0603_1608Metric, F.Cu at (119.5, 87.2)
- added R32: 562k, Resistor_SMD:R_0603_1608Metric, F.Cu at (78.8, 128.6)
- added R33: 0R, Resistor_SMD:R_0603_1608Metric, F.Cu at (173.5, 128.2)
- added R34: 0R, Resistor_SMD:R_0603_1608Metric, F.Cu at (164.7, 69.9)
- added R35: 0R, Resistor_SMD:R_0603_1608Metric, F.Cu at (84.2, 128.3)
- added R36: 200R, Resistor_SMD:R_0603_1608Metric, F.Cu at (154.9, 117.7)
- added R37: 200R, Resistor_SMD:R_0603_1608Metric, F.Cu at (171.0, 77.7)
- added R38: R_Small, Resistor_SMD:R_0603_1608Metric, F.Cu at (85.2, 121.0)
- added R39: 0402 RF 50 Ohm thin film, Resistor_SMD:R_0402_1005Metric, F.Cu at (131.5, 76.6)
- added R4: 10k, Resistor_SMD:R_0603_1608Metric, F.Cu at (94.8, 114.0)
- added R40: 500R, Resistor_SMD:R_0402_1005Metric, F.Cu at (163.8, 108.7)
- added R41: 500R, Resistor_SMD:R_0402_1005Metric, F.Cu at (170.5, 107.9)
- added R42: 500R, Resistor_SMD:R_0402_1005Metric, F.Cu at (164.6, 90.6)
- added R43: 500R, Resistor_SMD:R_0402_1005Metric, F.Cu at (170.0, 90.4)
- added R44: R_Small, Resistor_SMD:R_0603_1608Metric, F.Cu at (157.8, 101.1)
- added R45: R_Small, Resistor_SMD:R_0603_1608Metric, F.Cu at (158.1, 105.3)
- added R46: R_Small, Resistor_SMD:R_0603_1608Metric, F.Cu at (155.4, 102.0)
- added R47: R_Small, Resistor_SMD:R_0603_1608Metric, F.Cu at (155.1, 98.2)
- added R49: R_Small, Resistor_SMD:R_0603_1608Metric, F.Cu at (105.2, 110.6)
- added R5: 0R, Resistor_SMD:R_0603_1608Metric, F.Cu at (61.3, 189.1)
- added R50: 10k, Resistor_SMD:R_0603_1608Metric, F.Cu at (65.6, 93.4)
- added R51: 121k, Resistor_SMD:R_0603_1608Metric, F.Cu at (60.2, 95.4)
- added R52: 249k, Resistor_SMD:R_0603_1608Metric, F.Cu at (60.2, 101.8)
- added R53: 49k, Resistor_SMD:R_0603_1608Metric, F.Cu at (60.2, 105.2)
- added R54: 180k, Resistor_SMD:R_0603_1608Metric, F.Cu at (65.3, 181.6)
- added R55: 562k, Resistor_SMD:R_0603_1608Metric, F.Cu at (73.5, 69.2)
- added R56: 0R, Resistor_SMD:R_0603_1608Metric, F.Cu at (71.0, 65.6)
- added R57: R_Small, Resistor_SMD:R_0603_1608Metric, F.Cu at (68.5, 69.2)
- added R58: 10k, Resistor_SMD:R_0603_1608Metric, F.Cu at (66.4, 78.6)
- added R59: 33k, Resistor_SMD:R_0603_1608Metric, F.Cu at (60.4, 80.2)
- added R6: 0R, Resistor_SMD:R_0603_1608Metric, F.Cu at (61.3, 191.6)
- added R60: 249k, Resistor_SMD:R_0603_1608Metric, F.Cu at (60.4, 86.6)
- added R61: 49k, Resistor_SMD:R_0603_1608Metric, F.Cu at (60.4, 89.8)
- added R62: 0R, Resistor_SMD:R_0603_1608Metric, F.Cu at (117.4, 129.6)
- added R63: 0R, Resistor_SMD:R_0603_1608Metric, F.Cu at (117.4, 132.1)
- added R64: 0R, Resistor_SMD:R_0603_1608Metric, F.Cu at (117.4, 134.6)
- added R7: R_Small, Resistor_SMD:R_0603_1608Metric, F.Cu at (102.9, 113.4)
- added R8: 100R, Resistor_SMD:R_0603_1608Metric, F.Cu at (134.1, 114.4)
- added R9: 1.5R, Resistor_SMD:R_0603_1608Metric, F.Cu at (134.4, 108.5)
- added SW1: SW_Push, Button_Switch_SMD:SW_SPST_CK_KXT3, F.Cu at (79.5, 81.5)
- IC4: footprint LMX:QFN50P600X600X100-41N-D -> Package_DFN_QFN:QFN-40-1EP_6x6mm_P0.5mm_EP4.6x4.6mm
- Q1: footprint Package_TO_SOT_THT:TO-220-3_Horizontal_TabDown -> Package_TO_SOT_SMD:TO-252-2
- moved J5 189.1 mm to (211.3, 121.5), turned to 0 degrees
- moved J6 182.5 mm to (211.6, 75.7), turned to 0 degrees
- moved FL3 152.7 mm to (196.3, 121.1), turned to -90 degrees
- moved IC6 150.5 mm to (187.9, 121.0), turned to 180 degrees
- moved T2 150.5 mm to (177.7, 123.8), turned to -90 degrees
- moved IC7 148.5 mm to (191.8, 75.3), turned to 180 degrees
- moved FL4 142.1 mm to (197.2, 75.3)
- moved C55 138.2 mm to (187.1, 128.4), turned to 180 degrees
- moved T1 136.5 mm to (154.5, 124.0), turned to 90 degrees
- moved C57 132.0 mm to (183.5, 128.2), turned to 180 degrees
- moved T3 127.9 mm to (178.8, 74.3), turned to -90 degrees
- moved FL1 125.4 mm to (201.9, 121.3), turned to 180 degrees
- moved IC9 122.1 mm to (166.1, 124.2), turned to 90 degrees
- moved IC1 117.0 mm to (70.0, 187.1)
- moved IC2 117.0 mm to (75.4, 187.1)
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Connections:
- IC11 pad 4: VDDSMPS -> VCC_ADC
- IC5 pad 1: +12V -> BAT+
- IC5 pad 2: +12V -> BAT+
- IC5 pad 3: +12V -> BAT+
- IC5 pad 9: 5V_CLEAN -> Net-(IC5-OUTS)
- PS1 pad 10: Net-(PS1-AVIN) -> BAT+
- PS1 pad 11: Net-(PS1-AVIN) -> BAT+
- PS1 pad 12: Net-(PS1-AVIN) -> BAT+
- PS1 pad 13: Net-(PS1-AVIN) -> BAT+
- Q1 pad 1: +12V -> BAT+
- Q1 pad 3: 5V_CLEAN -> Net-(IC5-OUTS)
Routing:
- net BAT+: track 0.00 -> 72.4 mm
- net VSS: track 0.00 -> 53.2 mm, vias 0 -> 2
- net Net-(IC5-OUT): track 0.00 -> 32.7 mm, vias 0 -> 2
- net Net-(IC12-OUT): track 0.00 -> 31.5 mm, vias 0 -> 2
- net Net-(IC12-OUTS): track 0.00 -> 30.7 mm
- net Net-(IC14-OUTS): track 0.00 -> 30.7 mm
- net Net-(IC5-OUTS): track 0.00 -> 28.2 mm
- net Net-(IC14-OUT): track 0.00 -> 27.8 mm, vias 0 -> 5
- net Net-(PS2-FSW): track 0.00 -> 24.0 mm
- net Net-(IC12-SET): track 0.00 -> 21.1 mm
- net Net-(IC5-SET): track 0.00 -> 14.9 mm, vias 0 -> 2
- net Net-(IC14-SET): track 0.00 -> 13.9 mm, vias 0 -> 2
- net VDDSMPS: track 0.00 -> 11.0 mm, vias 0 -> 2
- net Net-(D5-A): track 0.00 -> 8.69 mm
- net Net-(IC12-PGFB): track 0.00 -> 4.20 mm, vias 0 -> 2
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Other:
- board outline added: 158.2 x 76.5 mm

Commit message: layout
Parts:
- moved H2 136.8 mm to (66.3, 144.1), turned to 0 degrees
- moved R35 45.4 mm to (129.1, 135.5), turned to 90 degrees
- moved SW1 39.1 mm to (104.5, 111.5)
- moved R27 34.8 mm to (154.6, 130.8)
- moved R34 31.9 mm to (148.7, 97.6), turned to 90 degrees
- moved C64 31.5 mm to (149.0, 93.0), turned to -90 degrees
- moved T2 31.4 mm to (153.1, 104.4), turned to 0 degrees
- moved R44 31.2 mm to (187.9, 92.7)
- moved R45 31.2 mm to (188.2, 96.9)
- moved R46 31.2 mm to (185.5, 93.6)
- moved C63 30.1 mm to (149.1, 89.2), turned to -90 degrees
- moved C55 29.2 mm to (157.9, 129.9), turned to -90 degrees
- moved C68 29.2 mm to (149.1, 85.7), turned to 90 degrees
- moved C60 29.0 mm to (158.8, 75.4)
- moved C57 28.9 mm to (154.6, 128.7)
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Connections:
- C72 pad 1: Net-(IC9-LOIP) -> Net-(IC9-LOIN)
- C73 pad 1: Net-(IC9-LOIN) -> Net-(IC9-LOIP)
- C77 pad 1: Net-(IC10-LOIP) -> Net-(IC10-LOIN)
- C78 pad 1: Net-(IC10-LOIN) -> Net-(IC10-LOIP)
- R23 pad 1: +12V -> 12V_CLEAN
Routing:
- net 5V_CLEAN: track 0.00 -> 109.1 mm, vias 0 -> 5
- net Net-(IC14-OUTS): track 30.7 -> 113.2 mm, vias 0 -> 2
- net Net-(PS1-FSW): track 0.00 -> 78.1 mm
- net Net-(IC12-OUTS): track 30.7 -> 101.9 mm, vias 0 -> 2
- net Net-(IC5-OUTS): track 28.2 -> 99.2 mm, vias 0 -> 2
- net RX2_SWITCH_BIT_2: track 0.00 -> 67.6 mm, vias 0 -> 1
- net RF_SWITCH_BIT_0: track 0.00 -> 53.5 mm, vias 0 -> 2
- net RF_SWITCH_BIT_1: track 0.00 -> 53.3 mm, vias 0 -> 2
- net VDDSMPS: track 11.0 -> 59.4 mm, vias 2 -> 3
- net RX1_SWITCH_BIT_0: track 0.00 -> 47.8 mm, vias 0 -> 1
- net RF_SWITCH_BIT_2: track 0.00 -> 47.5 mm, vias 0 -> 2
- net RX2_SWITCH_BIT_0: track 0.00 -> 45.4 mm, vias 0 -> 1
- net RX1_SWITCH_BIT_1: track 0.00 -> 44.7 mm, vias 0 -> 1
- net RX1_SWITCH_BIT_2: track 0.00 -> 41.7 mm, vias 0 -> 1
- net SWCLK: track 0.00 -> 41.5 mm
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Other:
- board size 158.2 x 76.5 mm -> 132.3 x 76.5 mm
- copper layers 2 -> 4

Commit message: update
Parts:
- removed C1: 2.2uF, Capacitor_SMD:C_0603_1608Metric
- removed C2: 100nF, Capacitor_SMD:C_0603_1608Metric
- removed TDK_HHM2952A1/auf_PCB1: DC4759J5020AHF-2, RF_Converter:Anaren_0805_2012Metric-6
- added C118: 100nF, Capacitor_SMD:C_0603_1608Metric, F.Cu at (106.3, 90.9)
- added C124: 100nF, Capacitor_SMD:C_0603_1608Metric, F.Cu at (95.0, 80.8)
- added C125: 100nF, Capacitor_SMD:C_0603_1608Metric, F.Cu at (91.6, 80.8)
- added C126: 100nF, Capacitor_SMD:C_0603_1608Metric, F.Cu at (88.2, 80.8)
- added C127: 100nF, Capacitor_SMD:C_0603_1608Metric, F.Cu at (82.4, 112.3)
- added C128: 100nF, Capacitor_SMD:C_0603_1608Metric, F.Cu at (88.3, 112.3)
- added C129: 100nF, Capacitor_SMD:C_0603_1608Metric, F.Cu at (91.5, 112.3)
- added C130: 100nF, Capacitor_SMD:C_0603_1608Metric, F.Cu at (98.5, 112.4)
- added C131: 100nF, Capacitor_SMD:C_0603_1608Metric, F.Cu at (106.3, 96.7)
- added C132: 100nF, Capacitor_SMD:C_0603_1608Metric, F.Cu at (106.3, 93.6)
- added C133: 100nF, Capacitor_SMD:C_0603_1608Metric, F.Cu at (98.4, 80.9)
- added C134: 100nF, Capacitor_SMD:C_0603_1608Metric, F.Cu at (74.8, 87.1)
- added C135: 100nF, Capacitor_SMD:C_0603_1608Metric, F.Cu at (100.2, 112.4)
- added C136: 100nF, Capacitor_SMD:C_0603_1608Metric, F.Cu at (106.2, 108.9)
- added C25: 100nF, Capacitor_SMD:C_0603_1608Metric, F.Cu at (74.7, 97.8)
- added C43: 100nF, Capacitor_SMD:C_0603_1608Metric, F.Cu at (74.9, 105.5)
- added C9: 100nF, Capacitor_SMD:C_0603_1608Metric, F.Cu at (74.7, 93.7)
- added U4: HHM2952A1, TDK:HHM2952A1, F.Cu at (123.3, 72.3)
- C38, C6, C8: footprint Capacitor_SMD:C_0805_2012Metric -> Capacitor_SMD:C_0603_1608Metric
- moved H2 113.6 mm to (179.6, 136.2)
- moved D3 53.3 mm to (135.4, 137.2), turned to 0 degrees
- moved C76 48.9 mm to (119.3, 107.3)
- moved R2 34.3 mm to (118.1, 135.5)
- moved R38 32.6 mm to (116.4, 135.5), turned to 90 degrees
- moved C14 27.7 mm to (117.0, 103.1), turned to 180 degrees
- moved C20 25.1 mm to (117.0, 104.7), turned to 180 degrees
- moved J3 24.2 mm to (81.2, 76.4), turned to 90 degrees
- moved R11 24.1 mm to (119.4, 103.9), turned to -90 degrees
- moved R7 23.2 mm to (114.6, 135.4)
- moved J7 21.2 mm to (106.3, 67.6)
- moved C107 17.7 mm to (167.0, 102.4), turned to -90 degrees
- moved R47 17.1 mm to (180.5, 91.6), turned to -90 degrees
- moved R49 15.9 mm to (107.5, 131.6), turned to 0 degrees
- moved R45 14.1 mm to (175.2, 91.4)
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Connections:
- C67 pad 1: Net-(PS1-FSW) -> Net-(D3-A)
- C76 pad 1: VCC_VCO -> Net-(D3-A)
- C80 pad 1: VCC_VCO -> Net-(D3-A)
- D3 pad 2: VCC_VCO -> Net-(D3-A)
- L6 pad 2: Net-(PS1-FSW) -> Net-(D3-A)
- PS1 pad 14: Net-(PS1-FSW) -> Net-(D3-A)
- PS1 pad 7: Net-(PS1-FSW) -> Net-(D3-A)
- R32 pad 2: Net-(PS1-FSW) -> Net-(D3-A)
- R35 pad 1: Net-(PS1-FSW) -> Net-(D3-A)
Routing:
- net SDOB: track 0.00 -> 124.6 mm, vias 0 -> 2
- net SDOC: track 0.00 -> 113.4 mm, vias 0 -> 3
- net SDOA: track 0.00 -> 90.4 mm, vias 0 -> 2
- net CSNOT: track 0.00 -> 89.6 mm, vias 0 -> 2
- net SCLK_ADC: track 0.00 -> 89.6 mm, vias 0 -> 2
- net VCC_ADC: track 0.00 -> 85.6 mm, vias 0 -> 4
- net Net-(PS1-FSW): track 78.1 -> 0.00 mm
- net Net-(IC14-OUTS): track 113.2 -> 42.0 mm, vias 2 -> 1
- net 12V_CLEAN: track 0.00 -> 56.6 mm, vias 0 -> 2
- net Net-(IC12-OUTS): track 101.9 -> 45.6 mm, vias 2 -> 1
- net SPLIT_TX: track 0.00 -> 54.6 mm
- net Net-(IC5-OUTS): track 99.2 -> 46.1 mm
- net 5V_CLEAN: track 109.1 -> 148.3 mm, vias 5 -> 7
- net VDDSMPS: track 59.4 -> 96.9 mm, vias 3 -> 0
- net Net-(IC9-QHI): track 0.00 -> 26.8 mm, vias 0 -> 2
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Other:
- board size 132.3 x 76.5 mm -> 125.6 x 75 mm
